Commit message: commit

File: src/aries/urdf/camera.xacro (robot description, xacro)
@@ -16,5 +16,5 @@
         <visual>
             <geometry>
-                <mesh filename="${mesh_location}/d435.dae"/>
+                <mesh filename="${mesh_location}/d435.stl"/>
             </geometry>
             <material name="red" />
@@ -22,5 +22,5 @@
         <collision>
             <geometry>
-                <mesh filename="${mesh_location}/d435.dae"/>
+                <mesh filename="${mesh_location}/d435.stl"/>
             </geometry>
         </collision>

File: src/aries/urdf/d435i.xacro (robot description, xacro)
@@ -37,12 +37,11 @@
         <visual>
             <geometry>
-                <mesh filename="${mesh_location}/d435.dae"/>
+                <mesh filename="${mesh_location}/d435.stl"/>
             </geometry>
             <material name="camera_aluminum"/>
         </visual>
         <collision>
-            <origin xyz="0 -0.0175 0" rpy="0 0 0"/>
             <geometry>
-                <box size="0.02505 0.090 0.025"/>
+                <mesh filename="${mesh_location}/d435.stl"/>
             </geometry>
         </collision>

File: src/aries/urdf/gripper_camera.xacro (robot description, xacro)
@@ -43,5 +43,5 @@
         <visual>
             <geometry>
-                <mesh filename="${mesh_location}/d435.dae"/>
+                <mesh filename="${mesh_location}/d435.stl"/>
             </geometry>
             <material name="camera_aluminum">
@@ -50,7 +50,6 @@
         </visual>
         <collision>
-            <origin xyz="0 -0.0175 0" rpy="0 0 0"/>
             <geometry>
-                <box size="0.02505 0.090 0.025"/>
+                <mesh filename="${mesh_location}/d435.stl"/>
             </geometry>
         </collision>
