Commit message: commit

File: src/aries/urdf/arm.xacro (robot description, xacro)
@@ -26,16 +26,16 @@
                     rpy="0 0 0" />
             <geometry>
-                <mesh filename="${mesh_location}/arm_base.stl" />
-            </geometry>
-            <material
-                name="">
-                <color rgba="1 1 1 1" />
-            </material>
-        </visual>
-        <collision>
-            <origin xyz="0 0 0"
-                    rpy="0 0 0" />
-            <geometry>
-                <mesh filename="${mesh_location}/arm_base.stl" />
+                <mesh filename="${mesh_location}/unused/arm_base.stl" />
+            </geometry>
+            <material
+                name="">
+                <color rgba="1 1 1 1" />
+            </material>
+        </visual>
+        <collision>
+            <origin xyz="0 0 0"
+                    rpy="0 0 0" />
+            <geometry>
+                <mesh filename="${mesh_location}/unused/arm_base.stl" />
             </geometry>
         </collision>
@@ -66,16 +66,16 @@
                     rpy="0 0 0" />
             <geometry>
-                <mesh filename="${mesh_location}/arm_shoulder.stl" />
-            </geometry>
-            <material
-                name="">
-                <color rgba="1 1 1 1" />
-            </material>
-        </visual>
-        <collision>
-            <origin xyz="0 0 0"
-                    rpy="0 0 0" />
-            <geometry>
-                <mesh filename="${mesh_location}/arm_shoulder.stl" />
+                <mesh filename="${mesh_location}/unused/arm_shoulder.stl" />
+            </geometry>
+            <material
+                name="">
+                <color rgba="1 1 1 1" />
+            </material>
+        </visual>
+        <collision>
+            <origin xyz="0 0 0"
+                    rpy="0 0 0" />
+            <geometry>
+                <mesh filename="${mesh_location}/unused/arm_shoulder.stl" />
             </geometry>
         </collision>
@@ -106,16 +106,16 @@
                     rpy="0 0 0" />
             <geometry>
-                <mesh filename="${mesh_location}/arm_elbow.stl" />
-            </geometry>
-            <material
-                name="">
-                <color rgba="1 1 1 1" />
-            </material>
-        </visual>
-        <collision>
-            <origin xyz="0 0 0"
-                    rpy="0 0 0" />
-            <geometry>
-                <mesh filename="${mesh_location}/arm_elbow.stl" />
+                <mesh filename="${mesh_location}/unused/arm_elbow.stl" />
+            </geometry>
+            <material
+                name="">
+                <color rgba="1 1 1 1" />
+            </material>
+        </visual>
+        <collision>
+            <origin xyz="0 0 0"
+                    rpy="0 0 0" />
+            <geometry>
+                <mesh filename="${mesh_location}/unused/arm_elbow.stl" />
             </geometry>
         </collision>
@@ -146,16 +146,16 @@
                     rpy="0 0 0" />
             <geometry>
-                <mesh filename="${mesh_location}/arm_wrist.stl" />
-            </geometry>
-            <material
-                name="">
-                <color rgba="1 1 1 1" />
-            </material>
-        </visual>
-        <collision>
-            <origin xyz="0 0 0"
-                    rpy="0 0 0" />
-            <geometry>
-                <mesh filename="${mesh_location}/arm_wrist.stl" />
+                <mesh filename="${mesh_location}/unused/arm_wrist.stl" />
+            </geometry>
+            <material
+                name="">
+                <color rgba="1 1 1 1" />
+            </material>
+        </visual>
+        <collision>
+            <origin xyz="0 0 0"
+                    rpy="0 0 0" />
+            <geometry>
+                <mesh filename="${mesh_location}/unused/arm_wrist.stl" />
             </geometry>
         </collision>

File: src/aries/urdf/igus_rebel2.urdf (robot description, URDF)
Before this commit: robot igus_rebel, 12 links, 11 joints
Links:
- link arm_base_link: geometry collision cylinder length=0.1 radius=0.09; visual mesh filename=file://$(find aries)/meshes/robolink_rebel2/rebel_6dof_03_v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
- link link1: geometry collision box size=0.1 0.03 0.1; visual mesh filename=file://$(find aries)/meshes/robolink_rebel2/rebel_6dof_03_v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
- link link2: geometry collision cylinder length=0.18 radius=0.06; visual mesh filename=file://$(find aries)/meshes/robolink_rebel2/rebel_6dof_03_v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
- link link3: geometry collision box size=0.1 0.03 0.1; visual mesh filename=file://$(find aries)/meshes/robolink_rebel2/rebel_6dof_03_v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
- link link4: geometry collision cylinder length=0.1 radius=0.05; visual mesh filename=file://$(find aries)/meshes/robolink_rebel2/rebel_6dof_03_v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
- link link5: geometry collision box size=0.1 0.03 0.1; visual mesh filename=file://$(find aries)/meshes/robolink_rebel2/rebel_6dof_03_v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
- link link6: geometry collision cylinder length=0.065 radius=0.04; visual mesh filename=file://$(find aries)/meshes/robolink_rebel2/rebel_6dof_03_v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
- link motor1: geometry collision cylinder length=0.065 radius=0.05; visual mesh filename=file://$(find aries)/meshes/robolink_rebel2/rebel_6dof_03_v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
- link motor2: geometry collision cylinder length=0.065 radius=0.05; visual mesh filename=file://$(find aries)/meshes/robolink_rebel2/rebel_6dof_03_v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
- link motor3: geometry collision cylinder length=0.065 radius=0.05; visual mesh filename=file://$(find aries)/meshes/robolink_rebel2/rebel_6dof_03_v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
- link motor4: geometry collision cylinder length=0.065 radius=0.05; visual mesh filename=file://$(find aries)/meshes/robolink_rebel2/rebel_6dof_03_v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
- link motor5: geometry collision cylinder length=0.065 radius=0.04; visual mesh filename=file://$(find aries)/meshes/robolink_rebel2/rebel_6dof_03_v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
