Commit message: commit

File: src/aries/urdf/common_properties.xacro (robot description, xacro)
@@ -21,5 +21,5 @@
   <xacro:property name="enable_mimic" value="true"/>
   <!-- Enable Lidar -->
-  <xacro:property name="enable_lidar" value="true"/>
+  <xacro:property name="enable_lidar" value="false"/>
   <!-- Keep real LiDAR frames/visuals in every robot description without
          automatically enabling the expensive Gazebo sensors. -->

Commit message: commit

File: src/aries/urdf/common_properties.xacro (robot description, xacro)
@@ -38,5 +38,5 @@
   <xacro:property name="enable_lidar_gazebo" value="false"/>
   <!-- Enable D435i -->
-  <xacro:property name="enable_D435i" value="false"/>
+  <xacro:property name="enable_D435i" value="true"/>
   <!-- Enable Gazebo extras used by the full robot description -->
   <xacro:property name="enable_full_robot_gazebo_extras" value="true"/>

File: src/aries/urdf/d435i.xacro (robot description, xacro)
@@ -14,8 +14,4 @@
     <xacro:property name="d435i_cam_depth_py" value="0.0175"/>
     <xacro:property name="d435i_cam_depth_pz" value="0.0125"/>
-    <!-- IMU Position Offset -->
-    <xacro:property name="d435i_imu_offset_x" value="-0.00174"/>
-    <xacro:property name="d435i_imu_offset_y" value="0.00552"/>
-    <xacro:property name="d435i_imu_offset_z" value="0.0176"/>
     <!-- Material definitions -->
     <material name="camera_aluminum">
@@ -47,8 +43,15 @@
             </geometry>
         </collision>
+        <!-- Uniform box of the collision dimensions (25.2 x 90 x 25 mm) at the
+             datasheet mass of the D435i. The previous 0.564 kg / 1e-3-scaled
+             tensor was neither the real camera nor consistent with the
+             identical gripper camera; both now derive from m/12*(a^2+b^2).
+             The COM sits at the collision box centroid, not at the link origin
+             (which is the bottom screw mount, on the front face). -->
         <inertial>
-            <mass value="0.564"/>
-            <origin xyz="0 0 0"/>
-            <inertia ixx="0.003881243" ixy="0.0" ixz="0.0" iyy="0.000498940" iyz="0.0" izz="0.003879257"/>
+            <mass value="0.072"/>
+            <origin xyz="-0.0126 0 0" rpy="0 0 0"/>
+            <inertia ixx="0.00005235" ixy="0.0" ixz="0.0"
+                     iyy="0.00000751" iyz="0.0" izz="0.00005236"/>
         </inertial>
     </link>
@@ -104,29 +107,7 @@
     </joint>
     <link name="camera_color_optical_frame"/>
-    <!-- Camera IMU sensor frames (accelerometer and gyroscope) -->
-    <joint name="camera_accel_joint" type="fixed">
-        <origin xyz="-0.00174 0.00552 0.0176" rpy="0 0 0"/>
-        <parent link="camera_link"/>
-        <child link="camera_accel_frame"/>
-    </joint>
-    <link name="camera_accel_frame"/>
-    <joint name="camera_accel_optical_joint" type="fixed">
-        <origin xyz="0 0 0" rpy="-1.5708 0 -1.5708"/>
-        <parent link="camera_accel_frame"/>
-        <child link="camera_accel_optical_frame"/>
-    </joint>
-    <link name="camera_accel_optical_frame"/>
-    <joint name="camera_gyro_joint" type="fixed">
-        <origin xyz="-0.00174 0.00552 0.0176" rpy="0 0 0"/>
-        <parent link="camera_link"/>
-        <child link="camera_gyro_frame"/>
-    </joint>
-    <link name="camera_gyro_frame"/>
-    <joint name="camera_gyro_optical_joint" type="fixed">
-        <origin xyz="0 0 0" rpy="-1.5708 0 -1.5708"/>
-        <parent link="camera_gyro_frame"/>
-        <child link="camera_gyro_optical_frame"/>
-    </joint>
-    <link name="camera_gyro_optical_frame"/>
+    <!-- The accel/gyro frames were removed with the IMU sensor: the D435i IMU is
+         not used anywhere in the stack, and the hardware driver is launched with
+         enable_gyro/enable_accel false, so it publishes no IMU frames either. -->
     <!-- Gazebo configuration for Ionic/ROS2 Jazzy -->
     <xacro:if value="${enable_D435i}">
@@ -141,5 +122,15 @@
             <!-- Color Camera Sensor - 15 Hz: nothing on the rover consumes this
                  stream faster, and every render sensor competes for GPU time with
-                 the gripper camera used for grasping. -->
+                 the gripper camera used for grasping.
+                 FOV/resolution are deliberately IDENTICAL to the depth sensor
+                 below. The RViz DepthCloud display (urdf_config.rviz) paints this
+                 image onto the depth image pixel-for-pixel, which is only valid
+                 when both share intrinsics; the depth sensor used to be 1.487 rad
+                 against this 1.211 rad, which mis-coloured the cloud by ~23 cm at
+                 the image edge at 1 m.
+                 gz_frame_id is depth_optical_frame, not color_optical_frame:
+                 Gazebo renders both sensors from camera_link, so declaring the
+                 color frame would apply a 15 mm offset that does not exist in
+                 simulation. Same reasoning as gripper_camera.xacro. -->
             <sensor name="camera_color" type="camera">
                 <camera name="camera">
@@ -164,5 +155,5 @@
                 <visualize>false</visualize>
                 <topic>camera/color/image_raw</topic>
-                <gz_frame_id>camera_color_optical_frame</gz_frame_id>
+                <gz_frame_id>camera_depth_optical_frame</gz_frame_id>
             </sensor>
             <!-- The infra1/infra2 render sensors were removed from simulation:
@@ -170,8 +161,9 @@
                  significant GPU time. The IR frames/links are kept for TF parity
                  with the hardware driver. -->
-            <!-- Depth Camera Sensor - 15 Hz (see color-sensor comment). -->
+            <!-- Depth Camera Sensor - 15 Hz, same intrinsics as the color sensor
+                 (see color-sensor comment for why they must match). -->
             <sensor name="camera_depth" type="depth_camera">
                 <camera name="camera">
-                    <horizontal_fov>1.487</horizontal_fov>
+                    <horizontal_fov>1.211</horizontal_fov>
                     <image>
                         <width>640</width>
@@ -183,8 +175,11 @@
                         <far>100</far>
                     </clip>
+                    <!-- 3 mm, the D435i datasheet figure and what the gripper
+                         camera uses. The old 0.100 m put +/-10 cm of noise on
+                         every pixel, which swamped the measurement entirely. -->
                     <noise>
                         <type>gaussian</type>
                         <mean>0.0</mean>
-                        <stddev>0.100</stddev>
+                        <stddev>0.003</stddev>
                     </noise>
                 </camera>
@@ -195,65 +190,7 @@
                 <gz_frame_id>camera_depth_optical_frame</gz_frame_id>
             </sensor>
-            <!-- IMU Sensor -->
-            <sensor name="camera_imu" type="imu">
-                <always_on>true</always_on>
-                <update_rate>400</update_rate>
-                <imu>
-                    <angular_velocity>
-                        <x>
-                            <noise type="gaussian">
-                                <mean>0.0</mean>
-                                <stddev>2e-4</stddev>
-                                <bias_mean>0.0000075</bias_mean>
-                                <bias_stddev>0.0000008</bias_stddev>
-                            </noise>
-                        </x>
-                        <y>
-                            <noise type="gaussian">
-                                <mean>0.0</mean>
-                                <stddev>2e-4</stddev>
-                                <bias_mean>0.0000075</bias_mean>
-                                <bias_stddev>0.0000008</bias_stddev>
-                            </noise>
-                        </y>
-                        <z>
-                            <noise type="gaussian">
-                                <mean>0.0</mean>
-                                <stddev>2e-4</stddev>
-                                <bias_mean>0.0000075</bias_mean>
-                                <bias_stddev>0.0000008</bias_stddev>
-                            </noise>
-                        </z>
-                    </angular_velocity>
-                    <linear_acceleration>
-                        <x>
-                            <noise type="gaussian">
-                                <mean>0.0</mean>
-                                <stddev>1.7e-2</stddev>
-                                <bias_mean>0.1</bias_mean>
-                                <bias_stddev>0.001</bias_stddev>
-                            </noise>
-                        </x>
-                        <y>
-                            <noise type="gaussian">
-                                <mean>0.0</mean>
-                                <stddev>1.7e-2</stddev>
-                                <bias_mean>0.1</bias_mean>
-                                <bias_stddev>0.001</bias_stddev>
-                            </noise>
-                        </y>
-                        <z>
-                            <noise type="gaussian">
-                                <mean>0.0</mean>
-                                <stddev>1.7e-2</stddev>
-                                <bias_mean>0.1</bias_mean>
-                                <bias_stddev>0.001</bias_stddev>
-                            </noise>
-                        </z>
-                    </linear_acceleration>
-                </imu>
-                <topic>camera/imu/data</topic>
-                <gz_frame_id>camera_gyro_optical_frame</gz_frame_id>
-            </sensor>
+            <!-- The IMU sensor was removed: nothing subscribes to it, it was
+                 bridged to ROS in no configuration, and the camera IMU is unused
+                 stack-wide (the rover has its own IMU). -->
         </gazebo>
     </xacro:if>

File: src/aries/urdf/gripper_camera.xacro (robot description, xacro)
@@ -9,11 +9,10 @@
           gripper_camera_left_ir_frame  / gripper_camera_left_ir_optical_frame
           gripper_camera_right_ir_frame / gripper_camera_right_ir_optical_frame
-          gripper_camera_accel_frame    / gripper_camera_accel_optical_frame
-          gripper_camera_gyro_frame     / gripper_camera_gyro_optical_frame
-        Gazebo sensor specs match Intel RealSense D435i datasheet
-          Color  69 deg H-FOV (1.204 rad), 1280x720, RGB_INT8,  30 Hz
-          Depth  85 deg H-FOV (1.487 rad), 1280x720, R_FLOAT32, 30 Hz, noise stddev 3 mm
-          Infra  85 deg H-FOV (1.487 rad),  640x480, L_INT8,    30 Hz
-          IMU    400 Hz, gyro + accel with realistic bias noise
+        Simulated sensors (matched to what the hardware driver is launched with
+        in aries_bringup/launch/aries_hardware.launch.py)
+          Color  69 deg H-FOV (1.204 rad), 640x480, RGB_INT8,   15 Hz
+          Depth  69 deg H-FOV (1.204 rad), 640x480, R_FLOAT32,  15 Hz, noise stddev 3 mm
+        No infra and no IMU: neither is used by anything in the stack, and each
+        extra render sensor costs real GPU time.
         ROS topics (bridged via gazebo_bridge.yaml)
           /gripper_camera/color/image_raw
@@ -21,10 +20,5 @@
           /gripper_camera/depth/image_rect_raw
           /gripper_camera/depth/camera_info
-          /gripper_camera/depth/image_rect_raw/points
-          /gripper_camera/infra1/image_rect_raw
-          /gripper_camera/infra1/camera_info
-          /gripper_camera/infra2/image_rect_raw
-          /gripper_camera/infra2/camera_info
-          /gripper_camera/imu/data
+          /gripper_camera/aligned_depth_to_color/image_raw  (alias of the depth image)
     -->
     <!-- Mount joint - attaches camera to gripper base -->
@@ -55,9 +49,14 @@
             </geometry>
         </collision>
+        <!-- Uniform box of the collision dimensions (25.2 x 90 x 25 mm) at the
+             datasheet mass, m/12*(a^2+b^2). The previous tensor was the rover
+             camera's scaled by 1e-3, which left it ~13x below the box value.
+             The COM sits at the collision box centroid, not at the link origin
+             (which is the bottom screw mount, on the front face). -->
         <inertial>
             <mass value="0.072"/>
-            <origin xyz="0 0 0"/>
-            <inertia ixx="0.000003881243" ixy="0.0" ixz="0.0"
-                     iyy="0.000000498940" iyz="0.0" izz="0.000003879257"/>
+            <origin xyz="-0.0126 0 0" rpy="0 0 0"/>
+            <inertia ixx="0.00005235" ixy="0.0" ixz="0.0"
+                     iyy="0.00000751" iyz="0.0" izz="0.00005236"/>
         </inertial>
     </link>
@@ -113,30 +112,7 @@
     </joint>
     <link name="gripper_camera_color_optical_frame"/>
-    <!-- IMU sensor frames -->
-    <!-- Offsets from official Intel D435i URDF (_d435i_imu_modules.urdf.xacro) -->
-    <joint name="gripper_camera_accel_joint" type="fixed">
-        <origin xyz="-0.01174 -0.00552 0.0051" rpy="0 0 0"/>
-        <parent link="gripper_camera_link"/>
-        <child link="gripper_camera_accel_frame"/>
-    </joint>
-    <link name="gripper_camera_accel_frame"/>
-    <joint name="gripper_camera_accel_optical_joint" type="fixed">
-        <origin xyz="0 0 0" rpy="-1.5708 0 -1.5708"/>
-        <parent link="gripper_camera_accel_frame"/>
-        <child link="gripper_camera_accel_optical_frame"/>
-    </joint>
-    <link name="gripper_camera_accel_optical_frame"/>
-    <joint name="gripper_camera_gyro_joint" type="fixed">
-        <origin xyz="-0.01174 -0.00552 0.0051" rpy="0 0 0"/>
-        <parent link="gripper_camera_link"/>
-        <child link="gripper_camera_gyro_frame"/>
-    </joint>
-    <link name="gripper_camera_gyro_frame"/>
-    <joint name="gripper_camera_gyro_optical_joint" type="fixed">
-        <origin xyz="0 0 0" rpy="-1.5708 0 -1.5708"/>
-        <parent link="gripper_camera_gyro_frame"/>
-        <child link="gripper_camera_gyro_optical_frame"/>
-    </joint>
-    <link name="gripper_camera_gyro_optical_frame"/>
+    <!-- The accel/gyro frames were removed with the IMU sensor: the D435i IMU is
+         not used anywhere in the stack, and the hardware driver is launched with
+         enable_gyro/enable_accel false, so it publishes no IMU frames either. -->
     <!-- Gazebo sensors -->
     <gazebo reference="gripper_camera_link">
@@ -212,65 +188,6 @@
             <gz_frame_id>gripper_camera_depth_optical_frame</gz_frame_id>
         </sensor>
-        <!-- IMU - D435i 400 Hz with realistic gyro + accel bias -->
-        <sensor name="gripper_camera_imu" type="imu">
-            <always_on>true</always_on>
-            <update_rate>400</update_rate>
-            <imu>
-                <angular_velocity>
-                    <x>
-                        <noise type="gaussian">
-                            <mean>0.0</mean>
-                            <stddev>2e-4</stddev>
-                            <bias_mean>0.0000075</bias_mean>
-                            <bias_stddev>0.0000008</bias_stddev>
-                        </noise>
-                    </x>
-                    <y>
-                        <noise type="gaussian">
-                            <mean>0.0</mean>
-                            <stddev>2e-4</stddev>
-                            <bias_mean>0.0000075</bias_mean>
-                            <bias_stddev>0.0000008</bias_stddev>
-                        </noise>
-                    </y>
-                    <z>
-                        <noise type="gaussian">
-                            <mean>0.0</mean>
-                            <stddev>2e-4</stddev>
-                            <bias_mean>0.0000075</bias_mean>
-                            <bias_stddev>0.0000008</bias_stddev>
-                        </noise>
-                    </z>
-                </angular_velocity>
-                <linear_acceleration>
-                    <x>
-                        <noise type="gaussian">
-                            <mean>0.0</mean>
-                            <stddev>1.7e-2</stddev>
-                            <bias_mean>0.1</bias_mean>
-                            <bias_stddev>0.001</bias_stddev>
-                        </noise>
-                    </x>
-                    <y>
-                        <noise type="gaussian">
-                            <mean>0.0</mean>
-                            <stddev>1.7e-2</stddev>
-                            <bias_mean>0.1</bias_mean>
-                            <bias_stddev>0.001</bias_stddev>
-                        </noise>
-                    </y>
-                    <z>
-                        <noise type="gaussian">
-                            <mean>0.0</mean>
-                            <stddev>1.7e-2</stddev>
-                            <bias_mean>0.1</bias_mean>
-                            <bias_stddev>0.001</bias_stddev>
-                        </noise>
-                    </z>
-                </linear_acceleration>
-            </imu>
-            <topic>gripper_camera/imu/data</topic>
-            <gz_frame_id>gripper_camera_gyro_optical_frame</gz_frame_id>
-        </sensor>
+        <!-- The IMU sensor was removed: nothing subscribes to it, and the
+             hardware driver runs with enable_gyro/enable_accel false. -->
     </gazebo>
 </robot>

File: src/aries/urdf/my_robot.urdf.xacro (robot description, xacro)
@@ -25,5 +25,4 @@
   <xacro:include filename="right_link.xacro"/>
   <xacro:include filename="lidar.xacro"/>
-  <!-- <xacro:include filename="camera.xacro" /> -->
   <xacro:include filename="d435i.xacro"/>
   <!-- <xacro:include filename="arm.xacro" /> -->
