Commit message: commit

File: src/aries/urdf/gripper_new.xacro (robot description, xacro)
@@ -368,4 +368,14 @@
         <origin xyz="0.0 0.0075 0.0" rpy="1.57 0 0"/>
     </joint>
+    <!-- Virtual TCP frame used as the IK tip: stable pinch center inside the
+         fingers. Finger z range is roughly 0.064-0.159 m from
+         arm_gripper_base_link; the bucket-jaw midpoint is ~0.22 m. -->
+    <xacro:property name="gripper_tcp_z" value="0.15"/>
+    <link name="gripper_tcp"/>
+    <joint name="gripper_tcp_joint" type="fixed">
+        <parent link="arm_gripper_base_link"/>
+        <child link="gripper_tcp"/>
+        <origin xyz="0.0 0.0 ${gripper_tcp_z}" rpy="0.0 0.0 0.0"/>
+    </joint>
     <!-- Gripper Camera (D435i) — defined in gripper_camera.xacro -->
     <xacro:include filename="gripper_camera.xacro" />

Commit message: commit

File: src/aries/urdf/gripper_new.xacro (robot description, xacro)
@@ -1,4 +1,12 @@
 <?xml version="1.0"?>
 <robot xmlns:xacro="http://www.ros.org/wiki/xacro">
+    <!-- Keep the nominal -1.57/0.07 commands inside Gazebo's physics limits.
+         When a commanded endpoint equals a DART hard stop, the linked mimic
+         joints can wedge there and refuse the following reverse command. Real
+         hardware retains its original physical limits. -->
+    <xacro:property name="gripper_joint_lower_limit"
+                    value="${-1.62 if gripper_hardware_protocol == 'gazebo' else -1.57}"/>
+    <xacro:property name="gripper_joint_upper_limit"
+                    value="${0.12 if gripper_hardware_protocol == 'gazebo' else 0.07}"/>
     <joint name="arm_gripper_base_joint" type="fixed">
         <parent link="link6"/>
@@ -75,5 +83,5 @@
         <origin xyz="-0.024 0.00838 0.090" rpy="-1.57 -1.57 0.0"/>
         <axis xyz="0 0 1"/>
-        <limit effort="500" velocity="1.0" lower="-1.57" upper="0.07"/>
+        <limit effort="500" velocity="1.0" lower="${gripper_joint_lower_limit}" upper="${gripper_joint_upper_limit}"/>
         <dynamics damping="10" friction="2"/>
     </joint>
@@ -115,5 +123,5 @@
         <origin xyz="0.024 0.00838 0.090" rpy="-1.57 -1.57 0.0"/>
         <axis xyz="0 0 -1"/>
-        <limit effort="500" velocity="1.0" lower="-1.57" upper="0.07"/>
+        <limit effort="500" velocity="1.0" lower="${gripper_joint_lower_limit}" upper="${gripper_joint_upper_limit}"/>
         <dynamics damping="10" friction="2"/>
         <mimic joint="gripper_gear_left_joint" multiplier="1.0" offset="0.0"/>
@@ -156,5 +164,5 @@
         <origin xyz="-0.012 0.00838 0.123" rpy="-1.57 -1.57 0.0"/>
         <axis xyz="0 0 1"/>
-        <limit effort="500" velocity="1.0" lower="-1.57" upper="0.07"/>
+        <limit effort="500" velocity="1.0" lower="${gripper_joint_lower_limit}" upper="${gripper_joint_upper_limit}"/>
         <dynamics damping="10" friction="2"/>
         <mimic joint="gripper_gear_left_joint" multiplier="1.0" offset="0.0"/>
@@ -210,5 +218,5 @@
         <origin xyz="0.012 0.00838 0.123" rpy="-1.57 -1.57 0.0"/>
         <axis xyz="0 0 -1"/>
-        <limit effort="500" velocity="1.0" lower="-1.57" upper="0.07"/>
+        <limit effort="500" velocity="1.0" lower="${gripper_joint_lower_limit}" upper="${gripper_joint_upper_limit}"/>
         <dynamics damping="10" friction="2"/>
         <mimic joint="gripper_gear_left_joint" multiplier="1.0" offset="0.0"/>

Commit message: commit

File: src/aries/urdf/gripper_new.xacro (robot description, xacro)
@@ -9,4 +9,8 @@
     <xacro:property name="gripper_joint_upper_limit"
                     value="${0.12 if gripper_hardware_protocol == 'gazebo' else 0.07}"/>
+    <!-- Physically swappable fingertip. finger_type is 'bucket', 'maintenance'
+         or 'probe'; each maps to gripper_<finger_type>.stl. All three share the
+         same mount pivots, so only the visual/collision mesh changes. -->
+    <xacro:property name="finger_mesh" value="gripper_${finger_type}.stl"/>
     <joint name="arm_gripper_base_joint" type="fixed">
         <parent link="link6"/>
@@ -252,16 +256,16 @@
                     rpy="0 0 0" />
             <geometry>
-                <mesh filename="${mesh_location}/gripper/gripper_bucket.stl" />
-            </geometry>
-            <material
-                name="">
-                <color rgba="1 1 1 1" />
-            </material>
-        </visual>
-        <collision>
-            <origin xyz="0 0 0"
-                    rpy="0 0 0" />
-            <geometry>
-                <mesh filename="${mesh_location}/gripper/gripper_bucket.stl" />
+                <mesh filename="${mesh_location}/gripper/${finger_mesh}" />
+            </geometry>
+            <material
+                name="">
+                <color rgba="1 1 1 1" />
+            </material>
+        </visual>
+        <collision>
+            <origin xyz="0 0 0"
+                    rpy="0 0 0" />
+            <geometry>
+                <mesh filename="${mesh_location}/gripper/${finger_mesh}" />
             </geometry>
         </collision>
@@ -306,16 +310,16 @@
                     rpy="0 0 0" />
             <geometry>
-                <mesh filename="${mesh_location}/gripper/gripper_bucket.stl" />
-            </geometry>
-            <material
-                name="">
-                <color rgba="1 1 1 1" />
-            </material>
-        </visual>
-        <collision>
-            <origin xyz="0 0 0"
-                    rpy="0 0 0" />
-            <geometry>
-                <mesh filename="${mesh_location}/gripper/gripper_bucket.stl" />
+                <mesh filename="${mesh_location}/gripper/${finger_mesh}" />
+            </geometry>
+            <material
+                name="">
+                <color rgba="1 1 1 1" />
+            </material>
+        </visual>
+        <collision>
+            <origin xyz="0 0 0"
+                    rpy="0 0 0" />
+            <geometry>
+                <mesh filename="${mesh_location}/gripper/${finger_mesh}" />
             </geometry>
         </collision>

File: src/aries/urdf/my_robot.urdf.xacro (robot description, xacro)
@@ -4,4 +4,7 @@
   <xacro:arg name="gripper_type" default="new"/>
   <xacro:property name="gripper_type" value="$(arg gripper_type)"/>
+  <!-- Swappable fingertip - 'bucket', 'maintenance', or 'probe' (new gripper only) -->
+  <xacro:arg name="finger_type" default="probe"/>
+  <xacro:property name="finger_type" value="$(arg finger_type)"/>
   <!-- Hardware protocol - 'mock_hardware', 'gazebo', or 'rebel' -->
   <xacro:arg name="hardware_protocol" default="gazebo"/>
