Commit message: commit

File: src/aries/urdf/igus_rebel2.control.xacro (robot description, xacro)
@@ -43,32 +43,39 @@
                     <state_interface name="velocity" />
                 </joint>
-                <!-- Mimic joints: driven by GazeboSimSystem to match gripper_gear_left_joint -->
+                <!-- The four-bar followers are READ ONLY here.
+                     They used to carry mimic/multiplier params as well, which
+                     coupled them a SECOND time: sdformat converts the URDF
+                     <mimic> tags in gripper_new.xacro into real SDF <mimic>
+                     constraints (confirmed with `gz sdf -p`), so DART already
+                     enforces q_follower = q_leader inside the solver. Adding
+                     the ros2_control mimic on top makes gz_ros2_control write
+                     a velocity command to each of the same five joints every
+                     cycle, so each DOF carries a hard kinematic constraint and
+                     an independent servo command that know nothing about each
+                     other, both with the joints' 500 N.m effort ceiling behind
+                     them. Two solvers arguing over one DOF is what tears a
+                     linkage apart on screen while every joint is individually
+                     "satisfied".
+                     Keep the constraint (it is solved with the dynamics and
+                     cannot drift) and drop the commands. The state interfaces
+                     stay so the followers still report their measured
+                     positions. -->
                 <joint name="gripper_gear_right_joint">
-                    <param name="mimic">gripper_gear_left_joint</param>
-                    <param name="multiplier">1.0</param>
                     <state_interface name="position" />
                     <state_interface name="velocity" />
                 </joint>
                 <joint name="gripper_link_left_joint">
-                    <param name="mimic">gripper_gear_left_joint</param>
-                    <param name="multiplier">1.0</param>
                     <state_interface name="position" />
                     <state_interface name="velocity" />
                 </joint>
                 <joint name="gripper_link_right_joint">
-                    <param name="mimic">gripper_gear_left_joint</param>
-                    <param name="multiplier">1.0</param>
                     <state_interface name="position" />
                     <state_interface name="velocity" />
                 </joint>
                 <joint name="gripper_bucket_left_joint">
-                    <param name="mimic">gripper_gear_left_joint</param>
-                    <param name="multiplier">1.0</param>
                     <state_interface name="position" />
                     <state_interface name="velocity" />
                 </joint>
                 <joint name="gripper_bucket_right_joint">
-                    <param name="mimic">gripper_gear_left_joint</param>
-                    <param name="multiplier">1.0</param>
                     <state_interface name="position" />
                     <state_interface name="velocity" />

Commit message: commit

File: src/aries/urdf/gripper_new.xacro (robot description, xacro)
@@ -13,21 +13,7 @@
          same mount pivots, so only the visual/collision mesh changes. -->
     <xacro:property name="finger_mesh" value="gripper_${finger_type}.stl"/>
-    <!-- Axial correction for where the fingertip actually sits on the bar.
-         The modelled tip sat 50 mm short of the real one: measured against
-         hardware with a probe actually gripped, the attached mesh landed
-         50.2 mm up the shaft from the real probe, with only 1.9 mm lateral and
-         1.3 deg of axis error - i.e. the error is purely along the finger, not
-         a pivot or bar-length problem (see attached_probe_axial_offset_m in
-         aries_vision_grasp/config/vision_grasp_params.yaml, which was the
-         workaround for exactly this). The modelled contact point sat at
-         z=0.220 where the real pinch is ~0.270.
-         Consequences of the old value: RViz drew the jaws 50 mm short, so they
-         could be touching a wheel in reality while the model showed clearance,
-         and MoveIt's collision model inherited the same blind spot.
-         Applied to the fingertip mesh only. The four-bar pivots are correct -
-         gripper_bucket_*_joint IS the gear bar's tip, which is what a four-bar
-         pivot means - so nothing about the linkage motion changes. Set to 0 to
-         restore the old geometry. If you measure flange-to-tip on the real
-         gripper (closed), the model should now read 397.2 mm; adjust here. -->
+    <!-- Keep the selected bucket/maintenance/probe mesh at its measured CAD
+         mounting position. A previous generic 50.2 mm shift was not valid for
+         the REBEL-6DOF-03 assembly and made every finger type incorrect. -->
     <xacro:property name="finger_axial_correction" value="0.0"/>
     <!-- Mass properties computed from each mesh by tetrahedron decomposition at
@@ -89,5 +75,5 @@
         <parent link="link6"/>
         <child link="arm_gripper_base_link"/>
-        <origin xyz="0.0 0.0 0.05223" rpy="0.0 0.0 3.14159"/>
+        <origin xyz="0.0 0.0 0.0522" rpy="0.0 0.0 3.141592653589793"/>
     </joint>
     <!--gripper base Link -->

Commit message: commit

File: src/aries/urdf/gripper_new.xacro (robot description, xacro)
@@ -100,4 +100,21 @@
             </geometry>
         </collision>
+        <!-- The four base pivot pins. The linkage is a DOUBLE-plate four-bar:
+             every bar is two plates 25 mm apart with the finger sandwiched
+             between them, and these 44 mm pins span the whole stack. Only the
+             far plate of each bar was ever modelled; the near plates are added
+             below on their own links. Geometry recovered from
+             gripper_missing_link.glb, placed by matching the reference CAD's
+             base to gripper_base.stl (0.0013 mm rms). Visual only - see the
+             note on gripper_gear_left_link. -->
+        <visual>
+            <origin xyz="0 0 0" rpy="0 0 0" />
+            <geometry>
+                <mesh filename="${mesh_location}/gripper/gripper_base_pins.stl" />
+            </geometry>
+            <material name="">
+                <color rgba="1 1 1 1" />
+            </material>
+        </visual>
     </link>
     <!--gripper_gear_left Link -->
@@ -123,4 +140,19 @@
             </geometry>
         </collision>
+        <!-- Near plate of this bar plus its tip pivot pin, at z = -25..-15 mm
+             in this frame (the modelled plate is z = 0..10, the finger rides
+             at -12.5 between them). Deliberately VISUAL ONLY: the modelled
+             plate and the finger already occupy this pivot's swept volume, so
+             adding collision here would mostly duplicate it. Add a matching
+             <collision> if you want the far side of the stack represented. -->
+        <visual>
+            <origin xyz="0 0 0" rpy="0 0 0" />
+            <geometry>
+                <mesh filename="${mesh_location}/gripper/gripper_gear_left_plate2.stl" />
+            </geometry>
+            <material name="">
+                <color rgba="1 1 1 1" />
+            </material>
+        </visual>
     </link>
     <joint name="gripper_gear_left_joint" type="revolute">
@@ -154,4 +186,14 @@
             </geometry>
         </collision>
+        <!-- Near plate + tip pin; mirror of gripper_gear_left_link. -->
+        <visual>
+            <origin xyz="0 0 0" rpy="0 0 0" />
+            <geometry>
+                <mesh filename="${mesh_location}/gripper/gripper_gear_right_plate2.stl" />
+            </geometry>
+            <material name="">
+                <color rgba="1 1 1 1" />
+            </material>
+        </visual>
     </link>
     <joint name="gripper_gear_right_joint" type="revolute">
@@ -186,4 +228,14 @@
             </geometry>
         </collision>
+        <!-- Near plate + tip pin of the follower bar. -->
+        <visual>
+            <origin xyz="0 0 0" rpy="0 0 0" />
+            <geometry>
+                <mesh filename="${mesh_location}/gripper/gripper_link_left_plate2.stl" />
+            </geometry>
+            <material name="">
+                <color rgba="1 1 1 1" />
+            </material>
+        </visual>
     </link>
     <joint name="gripper_link_left_joint" type="revolute">
@@ -237,4 +289,14 @@
             </geometry>
         </collision>
+        <!-- Near plate + tip pin; mirror of gripper_left_link. -->
+        <visual>
+            <origin xyz="0 0 0" rpy="0 0 0" />
+            <geometry>
+                <mesh filename="${mesh_location}/gripper/gripper_link_right_plate2.stl" />
+            </geometry>
+            <material name="">
+                <color rgba="1 1 1 1" />
+            </material>
+        </visual>
     </link>
     <joint name="gripper_link_right_joint" type="revolute">

File: src/aries/urdf/right_link.xacro (robot description, xacro)
@@ -123,5 +123,5 @@
             <origin xyz="0 0 0" rpy="${PI/2} 0 ${PI}"/>
             <geometry>
-                <mesh filename="${mesh_location}/R_2_Wheel_Link_v2.glb"/>
+                <mesh filename="${mesh_location}/R_3_Wheel_Link_v2.glb"/>
             </geometry>
         </visual>
@@ -129,5 +129,5 @@
             <origin xyz="0 0.035 0" rpy="${PI/2} 0 0"/>
             <geometry>
-                <mesh filename="${mesh_location}/R_2_Wheel_Link_v2.stl"/>
+                <mesh filename="${mesh_location}/R_3_Wheel_Link_v2.stl"/>
             </geometry>
         </collision>

Commit message: commit

File: src/aries/urdf/gripper_new.xacro (robot description, xacro)
@@ -39,4 +39,76 @@
     <xacro:property name="finger_iyz"
                     value="${-3.025e-07 if finger_type == 'probe' else (3.143e-06 if finger_type == 'bucket' else -1.008e-06)}"/>
+    <!-- Fingertip COLLISION is boxes, not the mesh, and it has to stay that way.
+         In this gz-sim 8.11 / DART-bullet stack a <mesh> collision generates NO
+         contacts against another <mesh> - bullet wraps both as concave GImpact
+         shapes and GImpact-vs-GImpact yields no manifold. Measured by dropping
+         probes on the maintenance panel's disconnect handle: a primitive box
+         rests on it at z=1.7844, this same fingertip STL falls through the
+         handle AND through the panel body to the ground. That is why the
+         fingers passed through everything they were asked to grasp.
+         The SDF escape hatch does not exist in this build. <convex_decomposition>
+         and <optimization> both pass `gz sdf -k` as "Valid", but only because
+         sdformat copies unknown elements through with a warning, and neither
+         changed the drop-test result. Do not put the mesh back on the strength
+         of `gz sdf -k`; re-run the drop test.
+         Three boxes per finger, z-bands tiling the mesh end to end so there is
+         no gap between them, x/y from a 400k-point surface sampling of each
+         STL. All three tips are symmetric about x, so only a width is needed.
+         The visual stays the real mesh. -->
+    <xacro:property name="finger_col_zlo"
+                    value="${-0.00496 if finger_type == 'probe' else (-0.00496 if finger_type == 'bucket' else -0.00494)}"/>
+    <xacro:property name="finger_col_zhi"
+                    value="${0.11959 if finger_type == 'probe' else (0.09488 if finger_type == 'bucket' else 0.11959)}"/>
+    <xacro:property name="finger_col0_x"
+                    value="${0.01500 if finger_type == 'probe' else (0.01500 if finger_type == 'bucket' else 0.01500)}"/>
+    <xacro:property name="finger_col0_ylo"
+                    value="${-0.00498 if finger_type == 'probe' else (-0.00497 if finger_type == 'bucket' else -0.00500)}"/>
+    <xacro:property name="finger_col0_yhi"
+                    value="${0.01819 if finger_type == 'probe' else (0.01563 if finger_type == 'bucket' else 0.01823)}"/>
+    <xacro:property name="finger_col1_x"
+                    value="${0.01840 if finger_type == 'probe' else (0.05000 if finger_type == 'bucket' else 0.01500)}"/>
+    <xacro:property name="finger_col1_ylo"
+                    value="${0.00224 if finger_type == 'probe' else (-0.02539 if finger_type == 'bucket' else 0.00228)}"/>
+    <xacro:property name="finger_col1_yhi"
+                    value="${0.01818 if finger_type == 'probe' else (0.01823 if finger_type == 'bucket' else 0.01822)}"/>
+    <xacro:property name="finger_col2_x"
+                    value="${0.03000 if finger_type == 'probe' else (0.05000 if finger_type == 'bucket' else 0.01500)}"/>
+    <xacro:property name="finger_col2_ylo"
+                    value="${-0.00273 if finger_type == 'probe' else (-0.02539 if finger_type == 'bucket' else -0.00255)}"/>
+    <xacro:property name="finger_col2_yhi"
+                    value="${0.01837 if finger_type == 'probe' else (0.01823 if finger_type == 'bucket' else 0.01852)}"/>
+    <xacro:property name="finger_col_dz" value="${(finger_col_zhi - finger_col_zlo) / 3}"/>
+    <!-- The bucket's last two bands are the scoop, and a box fills its bowl:
+         the proxy is SOLID where the real tip is a shell. Nothing in these
+         worlds is scooped as particles, so a conservative solid is the right
+         trade; if granular digging is ever simulated this tip needs a proper
+         three-box U instead. -->
+    <xacro:macro name="finger_collision_boxes">
+      <xacro:property name="band" value="0"/>
+      <collision name="tip_band0">
+        <origin xyz="0 ${(finger_col0_yhi + finger_col0_ylo) / 2}
+                       ${finger_col_zlo + finger_col_dz * 0.5 + finger_axial_correction}"
+                rpy="0 0 0"/>
+        <geometry>
+          <box size="${finger_col0_x} ${finger_col0_yhi - finger_col0_ylo} ${finger_col_dz}"/>
+        </geometry>
+      </collision>
+      <collision name="tip_band1">
+        <origin xyz="0 ${(finger_col1_yhi + finger_col1_ylo) / 2}
+                       ${finger_col_zlo + finger_col_dz * 1.5 + finger_axial_correction}"
+                rpy="0 0 0"/>
+        <geometry>
+          <box size="${finger_col1_x} ${finger_col1_yhi - finger_col1_ylo} ${finger_col_dz}"/>
+        </geometry>
+      </collision>
+      <collision name="tip_band2">
+        <origin xyz="0 ${(finger_col2_yhi + finger_col2_ylo) / 2}
+                       ${finger_col_zlo + finger_col_dz * 2.5 + finger_axial_correction}"
+                rpy="0 0 0"/>
+        <geometry>
+          <box size="${finger_col2_x} ${finger_col2_yhi - finger_col2_ylo} ${finger_col_dz}"/>
+        </geometry>
+      </collision>
+    </xacro:macro>
     <!-- Reusable inertial blocks. -->
     <xacro:macro name="gripper_inertial" params="mass cx cy cz ixx iyy izz ixy:=0 ixz:=0 iyz:=0">
@@ -344,11 +416,5 @@
             </material>
         </visual>
-        <collision>
-            <origin xyz="0 0 ${finger_axial_correction}"
-                    rpy="0 0 0" />
-            <geometry>
-                <mesh filename="${mesh_location}/gripper/${finger_mesh}" />
-            </geometry>
-        </collision>
+        <xacro:finger_collision_boxes/>
     </link>
     <!-- Local +Z here maps to base +Y (the plate-stack depth direction). The
@@ -416,11 +482,5 @@
             </material>
         </visual>
-        <collision>
-            <origin xyz="0 0 ${finger_axial_correction}"
-                    rpy="0 0 0" />
-            <geometry>
-                <mesh filename="${mesh_location}/gripper/${finger_mesh}" />
-            </geometry>
-        </collision>
+        <xacro:finger_collision_boxes/>
     </link>
     <!-- Mirror of gripper_bucket_left_joint; same inboard-face step sign. -->

File: src/aries/urdf/gripper_v2.xacro (robot description, xacro)
@@ -148,4 +148,91 @@
         </collision>
     </xacro:macro>
+    <!-- The FINGERTIPS are the exception to the macro above: their collision is
+         boxes, and it has to stay that way.
+         In this gz-sim 8.11 / DART-bullet stack a <mesh> collision generates NO
+         contacts against another <mesh>. Bullet wraps both as concave GImpact
+         shapes and GImpact-vs-GImpact yields no manifold. Measured by dropping
+         probes onto the maintenance panel's disconnect handle: a primitive box
+         comes to rest on it at z=1.7844, while a fingertip STL falls straight
+         through the handle AND through the panel body onto the ground. That is
+         why the gripper passed through everything it was asked to operate.
+         The SDF escape hatch does not exist in this build: <convex_decomposition>
+         and <optimization> both pass `gz sdf -k` as "Valid" - only because
+         sdformat copies unknown elements through with a warning - and neither
+         changed the drop test. Do not restore the mesh on the strength of
+         `gz sdf -k`; re-run the drop test.
+         Three boxes per tip, z-bands tiling the mesh end to end so there is no
+         gap, x/y from a 300k-point surface sampling of each STL. Left and right
+         are exact mirrors, so one set of numbers serves both with sx = +/-1.
+         The visual stays the real mesh. -->
+    <xacro:property name="finger_col0_sx"
+                    value="${0.0262 if finger_type == 'probe' else (0.0270 if finger_type == 'bucket' else 0.0261)}"/>
+    <xacro:property name="finger_col0_sy"
+                    value="${0.0150 if finger_type == 'probe' else (0.0150 if finger_type == 'bucket' else 0.0150)}"/>
+    <xacro:property name="finger_col0_sz"
+                    value="${0.0335 if finger_type == 'probe' else (0.0368 if finger_type == 'bucket' else 0.0331)}"/>
+    <xacro:property name="finger_col0_x"
+                    value="${0.00812 if finger_type == 'probe' else (0.00849 if finger_type == 'bucket' else 0.00803)}"/>
+    <xacro:property name="finger_col0_y"
+                    value="${0.0 if finger_type == 'probe' else (-0.00005 if finger_type == 'bucket' else 0.0)}"/>
+    <xacro:property name="finger_col0_z"
+                    value="${0.01180 if finger_type == 'probe' else (0.01346 if finger_type == 'bucket' else 0.01165)}"/>
+    <xacro:property name="finger_col1_sx"
+                    value="${0.0173 if finger_type == 'probe' else (0.0466 if finger_type == 'bucket' else 0.0174)}"/>
+    <xacro:property name="finger_col1_sy"
+                    value="${0.0300 if finger_type == 'probe' else (0.0500 if finger_type == 'bucket' else 0.0150)}"/>
+    <xacro:property name="finger_col1_sz"
+                    value="${0.0335 if finger_type == 'probe' else (0.0368 if finger_type == 'bucket' else 0.0331)}"/>
+    <xacro:property name="finger_col1_x"
+                    value="${0.01627 if finger_type == 'probe' else (0.00633 if finger_type == 'bucket' else 0.01588)}"/>
+    <xacro:property name="finger_col1_y"
+                    value="${0.0 if finger_type == 'probe' else (-0.00005 if finger_type == 'bucket' else 0.0)}"/>
+    <xacro:property name="finger_col1_z"
+                    value="${0.04525 if finger_type == 'probe' else (0.05023 if finger_type == 'bucket' else 0.04479)}"/>
+    <xacro:property name="finger_col2_sx"
+                    value="${0.0217 if finger_type == 'probe' else (0.0483 if finger_type == 'bucket' else 0.0216)}"/>
+    <xacro:property name="finger_col2_sy"
+                    value="${0.0300 if finger_type == 'probe' else (0.0500 if finger_type == 'bucket' else 0.0150)}"/>
+    <xacro:property name="finger_col2_sz"
+                    value="${0.0335 if finger_type == 'probe' else (0.0368 if finger_type == 'bucket' else 0.0331)}"/>
+    <xacro:property name="finger_col2_x"
+                    value="${0.02568 if finger_type == 'probe' else (0.00883 if finger_type == 'bucket' else 0.02522)}"/>
+    <xacro:property name="finger_col2_y"
+                    value="${0.0 if finger_type == 'probe' else (-0.00005 if finger_type == 'bucket' else 0.0)}"/>
+    <xacro:property name="finger_col2_z"
+                    value="${0.07870 if finger_type == 'probe' else (0.08699 if finger_type == 'bucket' else 0.07793)}"/>
+    <!-- The bucket's upper two bands are its scoop, and a box fills the bowl:
+         the proxy is SOLID where the real tip is a shell. Nothing in these
+         worlds is scooped as particles, so a conservative solid is the right
+         trade; granular digging would need a proper three-box U instead. -->
+    <xacro:macro name="finger_geometry" params="file sx">
+        <visual>
+            <origin xyz="0 0 0" rpy="0 0 0"/>
+            <geometry>
+                <mesh filename="${mesh_location}/gripper_v2/${file}"/>
+            </geometry>
+            <material name="">
+                <color rgba="1 1 1 1"/>
+            </material>
+        </visual>
+        <collision name="tip_band0">
+            <origin xyz="${sx * finger_col0_x} ${finger_col0_y} ${finger_col0_z}" rpy="0 0 0"/>
+            <geometry>
+                <box size="${finger_col0_sx} ${finger_col0_sy} ${finger_col0_sz}"/>
+            </geometry>
+        </collision>
+        <collision name="tip_band1">
+            <origin xyz="${sx * finger_col1_x} ${finger_col1_y} ${finger_col1_z}" rpy="0 0 0"/>
+            <geometry>
+                <box size="${finger_col1_sx} ${finger_col1_sy} ${finger_col1_sz}"/>
+            </geometry>
+        </collision>
+        <collision name="tip_band2">
+            <origin xyz="${sx * finger_col2_x} ${finger_col2_y} ${finger_col2_z}" rpy="0 0 0"/>
+            <geometry>
+                <box size="${finger_col2_sx} ${finger_col2_sy} ${finger_col2_sz}"/>
+            </geometry>
+        </collision>
+    </xacro:macro>
     <!-- Joint damping/friction, sized against the inertias above; see the long
          note in gripper_new.xacro for why they cannot be left at the 10/2 that
@@ -288,5 +375,5 @@
                                 ixx="${finger_ixx}" iyy="${finger_iyy}" izz="${finger_izz}"
                                 ixz="${finger_ixz}"/>
-        <xacro:gripper_mesh_geometry file="${finger_mesh_left}"/>
+        <xacro:finger_geometry file="${finger_mesh_left}" sx="1"/>
     </link>
     <joint name="gripper_bucket_left_joint" type="revolute">
@@ -304,5 +391,5 @@
                                 ixx="${finger_ixx}" iyy="${finger_iyy}" izz="${finger_izz}"
                                 ixz="${-finger_ixz}"/>
-        <xacro:gripper_mesh_geometry file="${finger_mesh_right}"/>
+        <xacro:finger_geometry file="${finger_mesh_right}" sx="-1"/>
     </link>
     <!-- Mirror of the left fingertip joint. Its parent already turns the other
