Commit message: commit

File: src/aries/urdf/left_link.xacro (robot description, xacro)
@@ -38,5 +38,5 @@
         <axis xyz="0 0 1"/>
         <limit lower="-0.226" upper="0.323" effort="1000" velocity="5"/>
-        <dynamics damping="50" friction="50"/>
+        <dynamics damping="500" friction="500" effort="1000"/>
     </joint>
     <!-- Left Wheel 1 -->

File: src/aries/urdf/right_link.xacro (robot description, xacro)
@@ -41,5 +41,5 @@
             <mimic joint="L_Rocker_Joint" multiplier="-1.0" offset="0.0"/>
         </xacro:if>
-        <dynamics damping="50" friction="50"/>
+        <dynamics damping="500" friction="500" effort="1000"/>
     </joint>
     <!-- Right Wheel 1 -->
