Commit message: commit

File: src/aries/urdf/aries_gazebo.xacro (robot description, xacro)
@@ -223,5 +223,5 @@
     </plugin>
   </gazebo>
-  <!-- Ground-truth odometry for debugging; DiffDrive owns /odom and /tf. -->
+  <!-- Ground-truth odometry drives the simulation EKF and corrected TF. -->
   <gazebo>
         <plugin filename="libgz-sim-odometry-publisher-system"
@@ -259,5 +259,7 @@
           <topic>/cmd_vel</topic>
           <odom_topic>/odom</odom_topic>
-          <tf_topic>/tf</tf_topic>
+          <!-- Keep wheel-integrated TF private to Gazebo. The simulation EKF
+               is the single ROS owner of odom -> base_footprint. -->
+          <tf_topic>/wheel_odom/tf</tf_topic>
           <child_frame_id>base_footprint</child_frame_id>
           <odom_publish_frequency>60</odom_publish_frequency>

File: src/aries/urdf/common_properties.xacro (robot description, xacro)
@@ -21,5 +21,5 @@
   <xacro:property name="enable_mimic" value="true"/>
   <!-- Enable Lidar -->
-  <xacro:property name="enable_lidar" value="false"/>
+  <xacro:property name="enable_lidar" value="true"/>
   <!-- Keep real LiDAR frames/visuals in every robot description without
          automatically enabling the expensive Gazebo sensors. -->

File: src/aries/urdf/lidar.xacro (robot description, xacro)
@@ -37,5 +37,8 @@
             <child link="Lidar_Scan_Link"/>
         </joint>
-        <gazebo reference="Lidar_Scan_Link">
+        <!-- Simulation rays are opt-in; physical bringup only needs the
+             links and fixed transforms above. -->
+        <xacro:if value="${enable_lidar_gazebo}">
+            <gazebo reference="Lidar_Scan_Link">
             <sensor name="gpu_lidar_points" type="gpu_lidar">
                 <pose>0 0 0 0 0 0</pose>
@@ -106,4 +109,5 @@
                 </sensor>
             </gazebo>
+        </xacro:if>
     </xacro:if>
 </robot>

File: src/aries/urdf/rover.urdf.xacro (robot description, xacro)
@@ -1,5 +1,9 @@
 <?xml version="1.0"?>
 <robot xmlns:xacro="http://www.ros.org/wiki/xacro" name="aries">
+  <xacro:arg name="enable_lidar_gazebo" default="false"/>
   <xacro:include filename="common_properties.xacro"/>
+  <xacro:property
+      name="enable_lidar_gazebo"
+      value="$(arg enable_lidar_gazebo)"/>
   <xacro:property name="enable_full_robot_gazebo_extras" value="false"/>
   <xacro:include filename="aries_gazebo.xacro"/>

Commit message: commit

File: src/aries/urdf/aries_gazebo.xacro (robot description, xacro)
@@ -95,6 +95,4 @@
     <maxVel>0.1</maxVel>
     <fdir1>1 0 0</fdir1>
-  </gazebo>
-  <gazebo reference="Lidar_Link">
   </gazebo>
   <!-- Gazebo Plugin for Joint State Publisher -->

File: src/aries/urdf/common_properties.xacro (robot description, xacro)
@@ -21,5 +21,5 @@
        hard-coded to 0.165, which left the wheels 41 mm BELOW base_footprint —
        everything treating that frame as ground (EKF, odom->base_footprint,
-       nav ground filtering, the LiDAR height) inherited that error.
+       nav ground filtering) inherited that error.
        Forward kinematics through the rocker/bogie chain puts the front and
        middle wheel centres 0.0964 m below base_link, so the base must stand
@@ -32,9 +32,4 @@
   <!-- Enable Mimic joints -->
   <xacro:property name="enable_mimic" value="true"/>
-  <!-- Enable Lidar -->
-  <xacro:property name="enable_lidar" value="true"/>
-  <!-- Keep real LiDAR frames/visuals in every robot description without
-         automatically enabling the expensive Gazebo sensors. -->
-  <xacro:property name="enable_lidar_gazebo" value="false"/>
   <!-- Enable D435i -->
   <xacro:property name="enable_D435i" value="true"/>

File: src/aries/urdf/my_robot.urdf.xacro (robot description, xacro)
@@ -25,5 +25,4 @@
   <xacro:include filename="left_link.xacro"/>
   <xacro:include filename="right_link.xacro"/>
-  <xacro:include filename="lidar.xacro"/>
   <xacro:include filename="d435i.xacro"/>
   <!-- <xacro:include filename="arm.xacro" /> -->

File: src/aries/urdf/rover.urdf.xacro (robot description, xacro)
@@ -1,9 +1,5 @@
 <?xml version="1.0"?>
 <robot xmlns:xacro="http://www.ros.org/wiki/xacro" name="aries">
-  <xacro:arg name="enable_lidar_gazebo" default="false"/>
   <xacro:include filename="common_properties.xacro"/>
-  <xacro:property
-      name="enable_lidar_gazebo"
-      value="$(arg enable_lidar_gazebo)"/>
   <xacro:property name="enable_full_robot_gazebo_extras" value="false"/>
   <xacro:include filename="aries_gazebo.xacro"/>
@@ -12,5 +8,4 @@
   <xacro:include filename="left_link.xacro"/>
   <xacro:include filename="right_link.xacro"/>
-  <xacro:include filename="lidar.xacro"/>
   <xacro:include filename="d435i.xacro"/>
 </robot>

Commit message: commit

File: src/aries/urdf/aries_gazebo.xacro (robot description, xacro)
@@ -43,6 +43,9 @@
   </gazebo>
   <gazebo reference="L_1_Wheel_Link">
-    <mu1>1.4</mu1>
-    <mu2>0.35</mu2>
+    <!-- Lugged tire: dry polymer tread has more grip than the soil can carry.
+         The Mars-yard surface therefore caps longitudinal traction at 0.60;
+         lower lateral grip permits physical scrub during skid steering. -->
+    <mu1>0.85</mu1>
+    <mu2>0.42</mu2>
     <kp>1000000.0</kp>
     <kd>100.0</kd>
@@ -52,6 +55,6 @@
   </gazebo>
   <gazebo reference="L_2_Wheel_Link">
-    <mu1>1.4</mu1>
-    <mu2>0.35</mu2>
+    <mu1>0.85</mu1>
+    <mu2>0.42</mu2>
     <kp>1000000.0</kp>
     <kd>100.0</kd>
@@ -61,6 +64,6 @@
   </gazebo>
   <gazebo reference="L_3_Wheel_Link">
-    <mu1>1.4</mu1>
-    <mu2>0.35</mu2>
+    <mu1>0.85</mu1>
+    <mu2>0.42</mu2>
     <kp>1000000.0</kp>
     <kd>100.0</kd>
@@ -70,6 +73,6 @@
   </gazebo>
   <gazebo reference="R_1_Wheel_Link">
-    <mu1>1.4</mu1>
-    <mu2>0.35</mu2>
+    <mu1>0.85</mu1>
+    <mu2>0.42</mu2>
     <kp>1000000.0</kp>
     <kd>100.0</kd>
@@ -79,6 +82,6 @@
   </gazebo>
   <gazebo reference="R_2_Wheel_Link">
-    <mu1>1.4</mu1>
-    <mu2>0.35</mu2>
+    <mu1>0.85</mu1>
+    <mu2>0.42</mu2>
     <kp>1000000.0</kp>
     <kd>100.0</kd>
@@ -88,6 +91,6 @@
   </gazebo>
   <gazebo reference="R_3_Wheel_Link">
-    <mu1>1.4</mu1>
-    <mu2>0.35</mu2>
+    <mu1>0.85</mu1>
+    <mu2>0.42</mu2>
     <kp>1000000.0</kp>
     <kd>100.0</kd>

File: src/aries/urdf/common_properties.xacro (robot description, xacro)
@@ -13,5 +13,9 @@
   <!-- Properties -->
   <xacro:property name="PI" value="3.1415926535897931"/>
-  <xacro:property name="wheel_mass" value="50"/>
+  <!-- Mass recovered from the exported wheel inertia tensor. For a wheel with
+       r = 0.110 m, I_axis = 0.0160988 kg m^2 = 1/2 m r^2 gives
+       m = 2.661 kg. The previous 50 kg placeholder made the six wheels alone
+       weigh 300 kg and produced non-physical normal/friction forces. -->
+  <xacro:property name="wheel_mass" value="2.661"/>
   <xacro:property name="wheel_radius" value="0.1100"/>
   <xacro:property name="wheel_thickness" value="0.070"/>

File: src/aries/urdf/left_link.xacro (robot description, xacro)
@@ -21,4 +21,7 @@
             <material name="silver"/>
         </visual>
+        <!-- Keep the exact CAD mesh for rendering, but use its measured outer
+             envelope for physics. Concave STL wheel collisions do not make
+             reliable contact with DART heightfields. -->
         <collision>
             <origin xyz="0 0 0" rpy="0 0 0"/>
@@ -59,5 +62,5 @@
             <origin xyz="0 0 0" rpy="${PI/2} 0 0"/>
             <geometry>
-                <mesh filename="${mesh_location}/L_1_Wheel_Link_v2.stl"/>
+                <cylinder radius="${wheel_radius}" length="${wheel_thickness}"/>
             </geometry>
         </collision>
@@ -92,5 +95,5 @@
             <origin xyz="0 0 0" rpy="${PI/2} 0 0"/>
             <geometry>
-                 <mesh filename="${mesh_location}/L_2_Wheel_Link_v2.stl"/>
+                 <cylinder radius="${wheel_radius}" length="${wheel_thickness}"/>
             </geometry>
         </collision>
@@ -125,5 +128,5 @@
             <origin xyz="0 0 0" rpy="${PI/2} 0 0"/>
             <geometry>
-                <mesh filename="${mesh_location}/L_3_Wheel_Link_v2.stl"/>
+                <cylinder radius="${wheel_radius}" length="${wheel_thickness}"/>
             </geometry>
         </collision>

File: src/aries/urdf/right_link.xacro (robot description, xacro)
@@ -21,4 +21,7 @@
             <material name="silver"/>
         </visual>
+        <!-- Keep the exact CAD mesh for rendering, but use its measured outer
+             envelope for physics. Concave STL wheel collisions do not make
+             reliable contact with DART heightfields. -->
         <collision>
             <origin xyz="0 0 0" rpy="0 0 0"/>
@@ -62,5 +65,5 @@
             <origin xyz="0 0 0" rpy="${PI/2} 0 0"/>
             <geometry>
-                <mesh filename="${mesh_location}/R_1_Wheel_Link_v2.stl"/>
+                <cylinder radius="${wheel_radius}" length="${wheel_thickness}"/>
             </geometry>
         </collision>
@@ -95,5 +98,5 @@
             <origin xyz="0 0 0" rpy="${PI/2} 0 0"/>
             <geometry>
-                <mesh filename="${mesh_location}/R_2_Wheel_Link_v2.stl"/>
+                <cylinder radius="${wheel_radius}" length="${wheel_thickness}"/>
             </geometry>
         </collision>
@@ -127,7 +130,7 @@
         </visual>
         <collision>
-            <origin xyz="0 0.035 0" rpy="${PI/2} 0 0"/>
-            <geometry>
-                <mesh filename="${mesh_location}/R_3_Wheel_Link_v2.stl"/>
+            <origin xyz="0 0 0" rpy="${PI/2} 0 0"/>
+            <geometry>
+                <cylinder radius="${wheel_radius}" length="${wheel_thickness}"/>
             </geometry>
         </collision>

Commit message: commit

File: src/aries/urdf/aries_gazebo.xacro (robot description, xacro)
@@ -166,4 +166,5 @@
             <joint_name>drill_motor_joint</joint_name>
             <joint_name>drill_container_joint</joint_name>
+            <joint_name>drill_bit_joint</joint_name>
         </plugin>
   </gazebo>
@@ -209,4 +210,18 @@
       <i_min>-20</i_min><i_max>20</i_max>
       <cmd_min>-100</cmd_min><cmd_max>100</cmd_max>
+    </plugin>
+    <!-- The auger spins, so this one is a VELOCITY controller, not a position
+         one: publish rad/s to the topic and a positive value turns it one way,
+         a negative value the other, indefinitely. Holding a spindle at an
+         angle, which is what JointPositionController would do, is not a thing
+         a drill does. It needs no holding controller either - the axis is
+         vertical and the bit's COM sits on it to within 46 um, so gravity
+         applies no torque about it. -->
+    <plugin filename="gz-sim-joint-controller-system"
+        name="gz::sim::systems::JointController">
+      <joint_name>drill_bit_joint</joint_name>
+      <topic>/model/aries/joint/drill_bit_joint/cmd_vel</topic>
+      <use_force_commands>true</use_force_commands>
+      <p_gain>2.0</p_gain><i_gain>0.2</i_gain>
     </plugin>
     <!-- <plugin filename="gz-sim-joint-position-controller-system"

File: src/aries/urdf/drill.xacro (robot description, xacro)
@@ -25,4 +25,9 @@
       the origin - and it is what the previous drill.xacro did for the fixed
       case. Inertial origins are therefore also in base_link coordinates.
+      drill_bit.glb is the ONE exception, and it has to be: it spins, and a
+      revolute axis passes through its link's origin, so a bit left in base_link
+      coordinates would orbit the rover's centreline half a metre away instead
+      of turning on itself. That mesh was re-datumed onto its own axis, so its
+      joint carries the axis position and its visual/inertial origins are local.
     -->
     <!-- ================================================================
@@ -114,15 +119,23 @@
          y = 0.0001) - 38 mm above the ground plane at the home pose, and it
          passes through the 50 mm bore in the base plate on the way down.
-         VISUAL ONLY, no <collision>, as specified. It shares the carriage's
-         frame through a fixed joint, so it feeds with the motor.
+         VISUAL ONLY, no <collision>, as specified. It hangs off the carriage,
+         so it feeds with the motor, and it spins on its own axis - see the
+         joint below.
          It still needs an <inertial>: 2.15 kg is a real fraction of the
-         carriage's swung mass, and a fixed-joint child with no inertial is
-         given a 1 kg unit-tensor default by the SDF converter, which would be
-         both wrong and silent. 274 cm^3 of steel at 7850 kg/m^3; the tensor
-         checks out against a slender rod, (1/12)mL^2 = 0.0546 vs 0.0538 here.
+         carriage's swung mass, and a link with no inertial is given a 1 kg
+         unit-tensor default by the SDF converter, which would be both wrong
+         and silent. 274 cm^3 of steel at 7850 kg/m^3. Both tensor entries that
+         matter check out: (1/12)mL^2 = 0.0546 against 0.0538 here for the
+         slender-rod terms, and izz = 1.024e-3 sits above a solid cylinder's
+         (1/2)mr^2 = 6.73e-4, which is what flighting carrying its mass out at
+         the rim should do.
+         Coordinates here are LOCAL to the bit, not base_link like every other
+         mesh in this file: drill_bit.glb was re-datumed onto the rotation axis
+         so the mesh origin is the axis. The COM lands 32 um / 46 um off it, so
+         the spinning mass is balanced and there is no wobble forcing.
          ================================================================ -->
     <link name="drill_bit_link">
         <inertial>
-            <origin xyz="-0.50948 0.00013 0.14368" rpy="0 0 0"/>
+            <origin xyz="0.000032 0.000046 0.143675" rpy="0 0 0"/>
             <mass value="2.1539"/>
             <inertia ixx="5.38379e-02" ixy="-5.78053e-07" ixz="-7.33246e-06"
@@ -136,8 +149,28 @@
         </visual>
     </link>
-    <joint name="drill_bit_joint" type="fixed">
+    <!--
+      Spindle rotation: continuous, so it turns either way without end, which is
+      what a drill that has to back out of a hole needs.
+      The origin is the one place in this file that is not 0 0 0, and it is not
+      optional. A revolute axis runs through the CHILD link's origin, so with
+      0 0 0 the bit would swing about base_link's centreline half a metre away
+      rather than turning on itself. x = -0.509508, y = 0.000085 is the axis
+      measured off the mesh, not eyeballed: the outer flighting holds
+      r_max = 25.000 mm about it at every height, and the 30 mm core agrees to
+      within 1 um. It is the same axis the lead screw is offset from and the
+      same one the base plate's 50 mm bore is centred on.
+      A continuous joint takes no lower/upper; effort and velocity are still
+      declared because ros2_control and gz both read them. 60 rad/s is ~570 rpm,
+      an upper bound for an auger of this size, and is a placeholder until the
+      drive is specified. Damping is deliberately low - this axis is meant to
+      spin freely, unlike the two feed axes.
+    -->
+    <joint name="drill_bit_joint" type="continuous">
         <parent link="drill_motor_link"/>
         <child link="drill_bit_link"/>
-        <origin xyz="0 0 0" rpy="0 0 0"/>
+        <origin xyz="-0.509508 0.000085 0" rpy="0 0 0"/>
+        <axis xyz="0 0 1"/>
+        <limit effort="20.0" velocity="60.0"/>
+        <dynamics damping="0.05" friction="0.02"/>
     </joint>
     <!-- ================================================================
