Commit message: commit

File: src/aries/urdf/d435i.xacro (robot description, xacro)
@@ -24,5 +24,5 @@
     <!-- Camera body, with origin at bottom screw mount -->
     <joint name="camera_joint" type="fixed">
-        <origin xyz="0.245 0.13 0.225" rpy="0 0 0"/>
+        <origin xyz="0.2756 0.0025 0.2535" rpy="0 0 0"/>
         <parent link="base_link"/>
         <child link="camera_bottom_screw_frame"/>

File: src/aries/urdf/igus_rebel_robot2.urdf.xacro (robot description, xacro)
@@ -9,5 +9,5 @@
     <parent link="base_link"/>
     <child link="arm_base_link"/>
-    <origin xyz="0.05121 0.0 0.2125" rpy="0.0 0.0 -0.10472"/>
+    <origin xyz="0.05121 0.0 0.2342" rpy="0.0 0.0 -0.10472"/>
   </joint>
 </robot>

File: src/aries/urdf/left_link.xacro (robot description, xacro)
@@ -40,5 +40,5 @@
     <link name="L_1_Wheel_Link">
         <inertial>
-            <origin xyz="0 0 0.0350608778434713" rpy="0 0 0"/>
+            <origin xyz="0 -0.0350608778434713 0" rpy="${-PI/2} 0 ${PI}"/>
             <mass value="${wheel_mass}"/>
             <inertia
@@ -51,5 +51,5 @@
         </inertial>
         <visual>
-            <origin xyz="0 0 0" rpy="0 0 0"/>
+            <origin xyz="0 0 0" rpy="${-PI/2} 0 ${PI}"/>
             <geometry>
                 <mesh filename="${mesh_location}/L_1_Wheel_Link.STL"/>
@@ -58,5 +58,5 @@
         </visual>
         <collision>
-            <origin xyz="0 0 0.035" rpy="0 0 0"/>
+            <origin xyz="0 -0.035 0" rpy="${PI/2} 0 0"/>
             <geometry>
                 <cylinder radius="${wheel_radius}" length="${wheel_thickness}"/>
@@ -64,10 +64,9 @@
         </collision>
     </link>
-    <!-- Left Wheel 1 Joint -->
     <joint name="L_1_Wheel_Joint" type="continuous">
-        <origin xyz="0.12754 0.1674 -0.0953" rpy="0 0 0"/>
+        <origin xyz="0.12754 0.1674 -0.0953" rpy="${-PI/2} 0 ${PI}"/>
         <parent link="L_Boggie_Link"/>
         <child link="L_1_Wheel_Link"/>
-        <axis xyz="0 0 -1"/>
+        <axis xyz="0 1 0"/>
         <dynamics damping="0.01" friction="0.01"/>
     </joint>
@@ -75,5 +74,5 @@
     <link name="L_2_Wheel_Link">
         <inertial>
-            <origin xyz="0 0 0.0350608778434713" rpy="0 0 0"/>
+            <origin xyz="0 -0.0350608778434713 0" rpy="${-PI/2} 0 ${PI}"/>
             <mass value="${wheel_mass}"/>
             <inertia
@@ -86,5 +85,5 @@
         </inertial>
         <visual>
-            <origin xyz="0 0 0" rpy="0 0 0"/>
+            <origin xyz="0 0 0" rpy="${-PI/2} 0 ${PI}"/>
             <geometry>
                 <mesh filename="${mesh_location}/L_2_Wheel_Link.STL"/>
@@ -93,5 +92,5 @@
         </visual>
         <collision>
-            <origin xyz="0 0 0.035" rpy="0 0 0"/>
+            <origin xyz="0 -0.035 0" rpy="${PI/2} 0 0"/>
             <geometry>
                 <cylinder radius="${wheel_radius}" length="${wheel_thickness}"/>
@@ -99,10 +98,9 @@
         </collision>
     </link>
-    <!-- Left Wheel 2 Joint -->
     <joint name="L_2_Wheel_Joint" type="continuous">
-        <origin xyz="-0.12754 0.1674 -0.0953" rpy="0 0 0"/>
+        <origin xyz="-0.12754 0.1674 -0.0953" rpy="${-PI/2} 0 ${PI}"/>
         <parent link="L_Boggie_Link"/>
         <child link="L_2_Wheel_Link"/>
-        <axis xyz="0 0 -1"/>
+        <axis xyz="0 1 0"/>
         <dynamics damping="0.01" friction="0.01"/>
     </joint>
@@ -110,5 +108,5 @@
     <link name="L_3_Wheel_Link">
         <inertial>
-            <origin xyz="0 0 0.0350608778434703" rpy="0 0 0"/>
+            <origin xyz="0 -0.0350608778434713 0" rpy="${-PI/2} 0 ${PI}"/>
             <mass value="${wheel_mass}"/>
             <inertia
@@ -121,5 +119,5 @@
         </inertial>
         <visual>
-            <origin xyz="0 0 0" rpy="0 0 0"/>
+            <origin xyz="0 0 0" rpy="${-PI/2} 0 ${PI}"/>
             <geometry>
                 <mesh filename="${mesh_location}/L_3_Wheel_Link.STL"/>
@@ -128,5 +126,5 @@
         </visual>
         <collision>
-            <origin xyz="0 0 0.035" rpy="0 0 0"/>
+            <origin xyz="0 -0.035 0" rpy="${PI/2} 0 0"/>
             <geometry>
                 <cylinder radius="${wheel_radius}" length="${wheel_thickness}"/>
@@ -136,8 +134,8 @@
     <!-- Left Wheel 3 Joint -->
     <joint name="L_3_Wheel_Joint" type="continuous">
-        <origin xyz="-0.2299 0.1602 -0.0953" rpy="0 0 0"/>
+        <origin xyz="-0.2299 0.1602 -0.0953" rpy="${-PI/2} 0 ${PI}"/>
         <parent link="L_Rocker_Link"/>
         <child link="L_3_Wheel_Link"/>
-        <axis xyz="0 0 -1"/>
+        <axis xyz="0 1 0"/>
         <dynamics damping="0.01" friction="0.01"/>
     </joint>

File: src/aries/urdf/lidar.xacro (robot description, xacro)
@@ -1,116 +1,103 @@
 <?xml version="1.0"?>
 <robot xmlns:xacro="http://www.ros.org/wiki/xacro">
-    <!-- Lidar Link -->
-     <xacro:if value="${enable_lidar}">
-      <!-- Measured mounting position on the physical rover. -->
-      <xacro:property name="lidar_mount_xyz" value="0.1947 -0.1126 0.27"/>
-      <link name="Lidar_Link">
-          <inertial>
-              <origin xyz="-0.000142451762346639 -0.0277692495246192 -2.91412068116337E-05" rpy="0 0 0"/>
-              <mass value="0.281890658237879"/>
-              <inertia
-                  ixx="0.000161112839542335"
-                  ixy="-1.13383824923403E-06"
-                  ixz="3.9288174866879E-07"
-                  iyy="0.000210368216440506"
-                  iyz="-2.31509209129161E-07"
-                  izz="0.000159257660338308"/>
-          </inertial>
-          <visual>
-              <origin xyz="0 0 0" rpy="0 0 0"/>
-              <geometry>
-                  <mesh filename="${mesh_location}/Lidar_Link.STL"/>
-              </geometry>
-              <material name="gray"/>
-          </visual>
-          <collision>
-              <origin xyz="0 0 0" rpy="0 0 0"/>
-              <geometry>
-                  <mesh filename="${mesh_location}/Lidar_Link.STL"/>
-              </geometry>
-          </collision>
-      </link>
-      <!-- Lidar Joint -->
-      <joint name="Lidar_Joint" type="fixed">
-          <!-- <origin xyz="0.1947 -0.1126 0.269999999999999" rpy="${PI/2} 0 ${PI/2}"/> -->
-          <origin xyz="${lidar_mount_xyz}" rpy="${PI/2} 0 ${PI/2}"/>
-          <parent link="base_link"/>
-          <child link="Lidar_Link"/>
-          <axis xyz="0 0 0"/>
-      </joint>
-      <!-- Base-aligned frame for the 2D LaserScan slice. -->
-      <link name="Lidar_Scan_Link"/>
-      <joint name="Lidar_Scan_Joint" type="fixed">
-          <origin xyz="${lidar_mount_xyz}" rpy="0 0 0"/>
-          <parent link="base_link"/>
-          <child link="Lidar_Scan_Link"/>
-      </joint>
-      <!-- Gazebo sensors are intentionally separate from the real LiDAR
-           frames so hardware descriptions do not start simulation sensors. -->
-      <xacro:if value="${enable_lidar_gazebo}">
-       <gazebo reference="Lidar_Link">
-        <sensor name="gpu_lidar" type="gpu_lidar">
-          <pose>0 0 0 0 0 0</pose>
-          <topic>/lidar</topic>
-          <update_rate>60</update_rate>
-          <ray>
-            <scan>
-              <horizontal>
-                <samples>1024</samples>
-                <resolution>1</resolution>
-                <min_angle>-3.14159</min_angle>
-                <max_angle> 3.14159</max_angle>
-              </horizontal>
-              <vertical>
-                <samples>1025</samples>
-                <resolution>1</resolution>
-                <min_angle>-3.14159</min_angle>
-                <max_angle> 3.14159</max_angle>
-              </vertical>
-            </scan>
-            <range>
-              <min>0.05</min>
-              <max>45.0</max>
-              <resolution>0.01</resolution>
-            </range>
-          </ray>
-          <gz_frame_id>Lidar_Link</gz_frame_id>
-          <always_on>1</always_on>
-          <visualize>true</visualize>
-        </sensor>
-       </gazebo>
-      <!-- Dedicated planar sensor for ROS LaserScan output. -->
-       <gazebo reference="base_link">
-        <sensor name="gpu_lidar_scan" type="gpu_lidar">
-          <pose>${lidar_mount_xyz} 0 0 0</pose>
-          <topic>/lidar_scan</topic>
-          <update_rate>60</update_rate>
-          <ray>
-            <scan>
-              <horizontal>
-                <samples>1024</samples>
-                <resolution>1</resolution>
-                <min_angle>-3.14159</min_angle>
-                <max_angle> 3.14159</max_angle>
-              </horizontal>
-              <vertical>
-                <samples>1</samples>
-                <resolution>1</resolution>
-                <min_angle>0.0</min_angle>
-                <max_angle>0.0</max_angle>
-              </vertical>
-            </scan>
-            <range>
-              <min>0.05</min>
-              <max>45.0</max>
-              <resolution>0.01</resolution>
-            </range>
-          </ray>
-          <gz_frame_id>Lidar_Scan_Link</gz_frame_id>
-          <always_on>1</always_on>
-          <visualize>false</visualize>
-        </sensor>
-       </gazebo>
-      </xacro:if>
+    <xacro:if value="${enable_lidar}">
+        <xacro:property name="lidar_mount_xyz" value="0.2 -0.105 0.2202"/>
+        <xacro:property name="sensor_height_offset" value="0.0628"/>
+        <link name="Lidar_Link">
+            <inertial>
+                <origin xyz="0 0 0" rpy="0 0 0"/>
+                <mass value="0.28"/>
+                <inertia ixx="0.0001" ixy="0" ixz="0" iyy="0.0001" iyz="0" izz="0.0001"/>
+            </inertial>
+            <visual>
+                <origin xyz="0.0 0.0 0.0" rpy="0 0 0"/>
+                <geometry>
+                    <mesh filename="${mesh_location}/picoscan_150.stl"/>
+                </geometry>
+                <material name="dark_grey">
+                    <color rgba="0.2 0.2 0.2 1.0"/>
+                </material>
+            </visual>
+            <collision>
+                <origin xyz="0.0 0.0 0.0" rpy="0 0 0"/>
+                <geometry>
+                    <mesh filename="${mesh_location}/picoscan_150.stl"/>
+                </geometry>
+            </collision>
+        </link>
+        <joint name="Lidar_Joint" type="fixed">
+            <origin xyz="${lidar_mount_xyz}" rpy="0 0 0"/>
+            <parent link="base_link"/>
+            <child link="Lidar_Link"/>
+        </joint>
+        <link name="Lidar_Scan_Link"/>
+        <joint name="Lidar_Scan_Joint" type="fixed">
+            <origin xyz="0 0 ${sensor_height_offset}" rpy="0 0 0"/>
+            <parent link="Lidar_Link"/>
+            <child link="Lidar_Scan_Link"/>
+        </joint>
+        <gazebo reference="Lidar_Scan_Link">
+            <sensor name="gpu_lidar_points" type="gpu_lidar">
+                <pose>0 0 0 0 0 0</pose>
+                <topic>/lidar</topic>
+                <update_rate>60</update_rate>
+                <ray>
+                    <scan>
+                    <horizontal>
+                        <samples>1024</samples>
+                        <resolution>1</resolution>
+                        <min_angle>-3.14159</min_angle>
+                        <max_angle> 3.14159</max_angle>
+                    </horizontal>
+                    <vertical>
+                        <samples>1025</samples>
+                        <resolution>1</resolution>
+                        <min_angle>-3.14159</min_angle>
+                        <max_angle> 3.14159</max_angle>
+                    </vertical>
+                    </scan>
+                    <range>
+                    <min>0.05</min>
+                    <max>45.0</max>
+                    <resolution>0.01</resolution>
+                    </range>
+                </ray>
+                <gz_frame_id>Lidar_Scan_Link</gz_frame_id>
+                <always_on>1</always_on>
+                <visualize>true</visualize>
+                </sensor>
+            </gazebo>
+            <!-- Dedicated planar sensor for ROS LaserScan output. -->
+            <gazebo reference="Lidar_Scan_Link">
+                <sensor name="gpu_lidar_scan" type="gpu_lidar">
+                <pose>0 0 0 0 0 0</pose>
+                <topic>/lidar_scan</topic>
+                <update_rate>60</update_rate>
+                <ray>
+                    <scan>
+                    <horizontal>
+                        <samples>1024</samples>
+                        <resolution>1</resolution>
+                        <min_angle>-3.14159</min_angle>
+                        <max_angle> 3.14159</max_angle>
+                    </horizontal>
+                    <vertical>
+                        <samples>1</samples>
+                        <resolution>1</resolution>
+                        <min_angle>0.0</min_angle>
+                        <max_angle>0.0</max_angle>
+                    </vertical>
+                    </scan>
+                    <range>
+                    <min>0.05</min>
+                    <max>45.0</max>
+                    <resolution>0.01</resolution>
+                    </range>
+                </ray>
+                <gz_frame_id>Lidar_Scan_Link</gz_frame_id>
+                <always_on>1</always_on>
+                <visualize>false</visualize>
+                </sensor>
+            </gazebo>
     </xacro:if>
 </robot>

File: src/aries/urdf/right_link.xacro (robot description, xacro)
@@ -43,5 +43,5 @@
     <link name="R_1_Wheel_Link">
         <inertial>
-            <origin xyz="0 0 0.0350608778434713" rpy="0 0 0"/>
+            <origin xyz="0 0.0350608778434713 0" rpy="${PI/2} 0 ${PI}"/>
             <mass value="${wheel_mass}"/>
             <inertia
@@ -54,5 +54,5 @@
             </inertial>
         <visual>
-            <origin xyz="0 0 0" rpy="0 0 0"/>
+            <origin xyz="0 0 0" rpy="${PI/2} 0 ${PI}"/>
             <geometry>
                 <mesh filename="${mesh_location}/R_1_Wheel_Link.STL"/>
@@ -61,5 +61,5 @@
         </visual>
         <collision>
-            <origin xyz="0 0 0.035" rpy="0 0 0"/>
+            <origin xyz="0 0.035 0" rpy="${PI/2} 0 0"/>
             <geometry>
                 <cylinder radius="${wheel_radius}" length="${wheel_thickness}"/>
@@ -67,10 +67,9 @@
         </collision>
     </link>
-    <!-- Right Wheel 1 Joint -->
     <joint name="R_1_Wheel_Joint" type="continuous">
-        <origin xyz="0.12754 -0.1674 -0.0953" rpy="0 0 0"/>
+        <origin xyz="0.12754 -0.1674 -0.0953" rpy="${PI/2} 0 ${PI}"/>
         <parent link="R_Boggie_Link"/>
         <child link="R_1_Wheel_Link"/>
-        <axis xyz="0 0 1"/>
+        <axis xyz="0 1 0"/>
         <dynamics damping="0.01" friction="0.01"/>
     </joint>
@@ -78,5 +77,5 @@
     <link name="R_2_Wheel_Link">
         <inertial>
-            <origin xyz="0 0 0.0350608778434713" rpy="0 0 0"/>
+            <origin xyz="0 0.0350608778434713 0" rpy="${PI/2} 0 ${PI}"/>
             <mass value="${wheel_mass}"/>
             <inertia
@@ -89,5 +88,5 @@
         </inertial>
         <visual>
-            <origin xyz="0 0 0" rpy="0 0 0"/>
+            <origin xyz="0 0 0" rpy="${PI/2} 0 ${PI}"/>
             <geometry>
                 <mesh filename="${mesh_location}/R_2_Wheel_Link.STL"/>
@@ -96,5 +95,5 @@
         </visual>
         <collision>
-            <origin xyz="0 0 0.035" rpy="0 0 0"/>
+            <origin xyz="0 0.035 0" rpy="${PI/2} 0 0"/>
             <geometry>
                 <cylinder radius="${wheel_radius}" length="${wheel_thickness}"/>
@@ -104,8 +103,8 @@
     <!-- Right Wheel 2 Joint -->
     <joint name="R_2_Wheel_Joint" type="continuous">
-        <origin xyz="-0.12754 -0.1674 -0.0953" rpy="0 0 0"/>
+        <origin xyz="-0.12754 -0.1674 -0.0953" rpy="${PI/2} 0 ${PI}"/>
         <parent link="R_Boggie_Link"/>
         <child link="R_2_Wheel_Link"/>
-        <axis xyz="0 0 1"/>
+        <axis xyz="0 1 0"/>
         <dynamics damping="0.01" friction="0.01"/>
     </joint>
@@ -113,5 +112,5 @@
     <link name="R_3_Wheel_Link">
         <inertial>
-            <origin xyz="0 0 0.0350608778434713" rpy="0 0 0"/>
+            <origin xyz="0 0.0350608778434713 0" rpy="${PI/2} 0 ${PI}"/>
             <mass value="${wheel_mass}"/>
             <inertia
@@ -124,5 +123,5 @@
         </inertial>
         <visual>
-            <origin xyz="0 0 0" rpy="0 0 0"/>
+            <origin xyz="0 0 0" rpy="${PI/2} 0 ${PI}"/>
             <geometry>
                 <mesh filename="${mesh_location}/R_3_Wheel_Link.STL"/>
@@ -131,5 +130,5 @@
         </visual>
         <collision>
-            <origin xyz="0 0 0.035" rpy="0 0 0"/>
+            <origin xyz="0 0.035 0" rpy="${PI/2} 0 0"/>
             <geometry>
                 <cylinder radius="${wheel_radius}" length="${wheel_thickness}"/>
@@ -139,8 +138,8 @@
     <!-- Right Wheel 3 Joint -->
     <joint name="R_3_Wheel_Joint" type="continuous">
-        <origin xyz="-0.2299 -0.1602 -0.0953" rpy="0 0 0"/>
+        <origin xyz="-0.2299 -0.1602 -0.0953" rpy="${PI/2} 0 ${PI}"/>
         <parent link="R_Rocker_Link"/>
         <child link="R_3_Wheel_Link"/>
-        <axis xyz="0 0 1"/>
+        <axis xyz="0 1 0"/>
         <dynamics damping="0.01" friction="0.01"/>
     </joint>
