Commit message: commit

File: src/aries/urdf/d435i.xacro (robot description, xacro)
@@ -19,16 +19,16 @@
     </material>
     <!-- Camera body, with origin at bottom screw mount -->
-    <joint name="camera_joint" type="fixed">
+    <joint name="rover_camera_joint" type="fixed">
         <origin xyz="0.2608 0.000023 0.2535" rpy="0 0 0"/>
         <parent link="base_link"/>
-        <child link="camera_bottom_screw_frame"/>
+        <child link="rover_camera_bottom_screw_frame"/>
     </joint>
-    <link name="camera_bottom_screw_frame"/>
-    <joint name="camera_link_joint" type="fixed">
+    <link name="rover_camera_bottom_screw_frame"/>
+    <joint name="rover_camera_link_joint" type="fixed">
         <origin xyz="0 0 0" rpy="0 0 0"/>
-        <parent link="camera_bottom_screw_frame"/>
-        <child link="camera_link"/>
+        <parent link="rover_camera_bottom_screw_frame"/>
+        <child link="rover_camera_link"/>
     </joint>
-    <link name="camera_link">
+    <link name="rover_camera_link">
         <visual>
             <geometry>
@@ -57,54 +57,54 @@
     </link>
     <!-- Camera depth sensor frames -->
-    <joint name="camera_depth_joint" type="fixed">
+    <joint name="rover_camera_depth_joint" type="fixed">
         <origin xyz="0 0 0" rpy="0 0 0"/>
-        <parent link="camera_link"/>
-        <child link="camera_depth_frame"/>
+        <parent link="rover_camera_link"/>
+        <child link="rover_camera_depth_frame"/>
     </joint>
-    <link name="camera_depth_frame"/>
-    <joint name="camera_depth_optical_joint" type="fixed">
+    <link name="rover_camera_depth_frame"/>
+    <joint name="rover_camera_depth_optical_joint" type="fixed">
         <origin xyz="0 0 0" rpy="-1.5708 0 -1.5708"/>
-        <parent link="camera_depth_frame"/>
-        <child link="camera_depth_optical_frame"/>
+        <parent link="rover_camera_depth_frame"/>
+        <child link="rover_camera_depth_optical_frame"/>
     </joint>
-    <link name="camera_depth_optical_frame"/>
+    <link name="rover_camera_depth_optical_frame"/>
     <!-- Camera IR sensor frames -->
-    <joint name="camera_left_ir_joint" type="fixed">
+    <joint name="rover_camera_left_ir_joint" type="fixed">
         <origin xyz="0 0.0 0" rpy="0 0 0"/>
-        <parent link="camera_depth_frame"/>
-        <child link="camera_left_ir_frame"/>
+        <parent link="rover_camera_depth_frame"/>
+        <child link="rover_camera_left_ir_frame"/>
     </joint>
-    <link name="camera_left_ir_frame"/>
-    <joint name="camera_left_ir_optical_joint" type="fixed">
+    <link name="rover_camera_left_ir_frame"/>
+    <joint name="rover_camera_left_ir_optical_joint" type="fixed">
         <origin xyz="0 0 0" rpy="-1.5708 0 -1.5708"/>
-        <parent link="camera_left_ir_frame"/>
-        <child link="camera_left_ir_optical_frame"/>
+        <parent link="rover_camera_left_ir_frame"/>
+        <child link="rover_camera_left_ir_optical_frame"/>
     </joint>
-    <link name="camera_left_ir_optical_frame"/>
-    <joint name="camera_right_ir_joint" type="fixed">
+    <link name="rover_camera_left_ir_optical_frame"/>
+    <joint name="rover_camera_right_ir_joint" type="fixed">
         <origin xyz="0 -0.050 0" rpy="0 0 0"/>
-        <parent link="camera_depth_frame"/>
-        <child link="camera_right_ir_frame"/>
+        <parent link="rover_camera_depth_frame"/>
+        <child link="rover_camera_right_ir_frame"/>
     </joint>
-    <link name="camera_right_ir_frame"/>
-    <joint name="camera_right_ir_optical_joint" type="fixed">
+    <link name="rover_camera_right_ir_frame"/>
+    <joint name="rover_camera_right_ir_optical_joint" type="fixed">
         <origin xyz="0 0 0" rpy="-1.5708 0 -1.5708"/>
-        <parent link="camera_right_ir_frame"/>
-        <child link="camera_right_ir_optical_frame"/>
+        <parent link="rover_camera_right_ir_frame"/>
+        <child link="rover_camera_right_ir_optical_frame"/>
     </joint>
-    <link name="camera_right_ir_optical_frame"/>
+    <link name="rover_camera_right_ir_optical_frame"/>
     <!-- Camera color sensor frames -->
-    <joint name="camera_color_joint" type="fixed">
+    <joint name="rover_camera_color_joint" type="fixed">
         <origin xyz="0 0.015 0" rpy="0 0 0"/>
-        <parent link="camera_depth_frame"/>
-        <child link="camera_color_frame"/>
+        <parent link="rover_camera_depth_frame"/>
+        <child link="rover_camera_color_frame"/>
     </joint>
-    <link name="camera_color_frame"/>
-    <joint name="camera_color_optical_joint" type="fixed">
+    <link name="rover_camera_color_frame"/>
+    <joint name="rover_camera_color_optical_joint" type="fixed">
         <origin xyz="0 0 0" rpy="-1.5708 0 -1.5708"/>
-        <parent link="camera_color_frame"/>
-        <child link="camera_color_optical_frame"/>
+        <parent link="rover_camera_color_frame"/>
+        <child link="rover_camera_color_optical_frame"/>
     </joint>
-    <link name="camera_color_optical_frame"/>
+    <link name="rover_camera_color_optical_frame"/>
     <!-- The accel/gyro frames were removed with the IMU sensor: the D435i IMU is
          not used anywhere in the stack, and the hardware driver is launched with
@@ -112,5 +112,5 @@
     <!-- Gazebo configuration for Ionic/ROS2 Jazzy -->
     <xacro:if value="${enable_D435i}">
-        <gazebo reference="camera_link">
+        <gazebo reference="rover_camera_link">
             <self_collide>0</self_collide>
             <enable_wind>0</enable_wind>
@@ -130,9 +130,9 @@
                  the image edge at 1 m.
                  gz_frame_id is depth_optical_frame, not color_optical_frame:
-                 Gazebo renders both sensors from camera_link, so declaring the
+                 Gazebo renders both sensors from rover_camera_link, so declaring the
                  color frame would apply a 15 mm offset that does not exist in
                  simulation. Same reasoning as gripper_camera.xacro. -->
-            <sensor name="camera_color" type="camera">
-                <camera name="camera">
+            <sensor name="rover_camera_color" type="camera">
+                <camera name="rover_camera">
                     <horizontal_fov>1.211</horizontal_fov>
                     <image>
@@ -154,6 +154,6 @@
                 <update_rate>15</update_rate>
                 <visualize>false</visualize>
-                <topic>camera/color/image_raw</topic>
-                <gz_frame_id>camera_depth_optical_frame</gz_frame_id>
+                <topic>rover_camera/color/image_raw</topic>
+                <gz_frame_id>rover_camera_depth_optical_frame</gz_frame_id>
             </sensor>
             <!-- The infra1/infra2 render sensors were removed from simulation:
@@ -163,6 +163,6 @@
             <!-- Depth Camera Sensor - 15 Hz, same intrinsics as the color sensor
                  (see color-sensor comment for why they must match). -->
-            <sensor name="camera_depth" type="depth_camera">
-                <camera name="camera">
+            <sensor name="rover_camera_depth" type="depth_camera">
+                <camera name="rover_camera">
                     <horizontal_fov>1.211</horizontal_fov>
                     <image>
@@ -187,6 +187,6 @@
                 <update_rate>15</update_rate>
                 <visualize>false</visualize>
-                <topic>camera/depth/image_rect_raw</topic>
-                <gz_frame_id>camera_depth_optical_frame</gz_frame_id>
+                <topic>rover_camera/depth/image_rect_raw</topic>
+                <gz_frame_id>rover_camera_depth_optical_frame</gz_frame_id>
             </sensor>
             <!-- The IMU sensor was removed: nothing subscribes to it, it was
