Commit message: commit

File: src/aries/urdf/gripper_camera.xacro (robot description, xacro)
@@ -30,5 +30,5 @@
     <!-- Mount joint - attaches camera to gripper base -->
     <joint name="gripper_camera_joint" type="fixed">
-        <origin xyz="0.0 0.045 0.035" rpy="0 -1.57 -1.57"/>
+        <origin xyz="0.0 0.047439 0.035208" rpy="0 -1.57 -1.57"/>
         <parent link="arm_gripper_base_link"/>
         <child link="gripper_camera_bottom_screw_frame"/>

Commit message: commit

File: src/aries/urdf/gripper_camera.xacro (robot description, xacro)
@@ -128,6 +128,6 @@
              vision_grasp_node indexes the depth image with color-image pixel
              coordinates. That is only geometrically valid when both cameras share the
-             same intrinsics. 15 Hz keeps the render-sensor load low; the vision node
-             only detects at 4 Hz and MoveIt's octomap updater is capped at 5 Hz. -->
+             same intrinsics. 15 Hz keeps the render-sensor load low while still
+             providing a responsive colored DepthCloud. -->
         <sensor name="gripper_camera_color" type="camera">
             <camera name="gripper_camera">

File: src/aries/urdf/gripper_v2.xacro (robot description, xacro)
@@ -63,4 +63,13 @@
     <xacro:property name="gripper_joint_upper_limit"
                     value="${0.12 if gripper_hardware_protocol == 'gazebo' else 0.07}"/>
+    <!-- The fingertip joints mimic the driver with multiplier -1.0, so their
+         limits must be transformed by the same relation.  Reusing the driver
+         limits makes every open pose invalid in MoveIt: driver q=-1.57 maps
+         to fingertip q=+1.57, which used to exceed the fingertip's +0.12
+         Gazebo limit. -->
+    <xacro:property name="gripper_bucket_joint_lower_limit"
+                    value="${-gripper_joint_upper_limit}"/>
+    <xacro:property name="gripper_bucket_joint_upper_limit"
+                    value="${-gripper_joint_lower_limit}"/>
     <!-- ZERO POSE.  The bars sit 11.3428 deg off the gripper axis at q = 0,
          which is the one free choice in the whole model: the CAD snapshot is a
@@ -287,5 +296,5 @@
         <axis xyz="0 1 0"/>
         <limit effort="500" velocity="1.0"
-               lower="${gripper_joint_lower_limit}" upper="${gripper_joint_upper_limit}"/>
+               lower="${gripper_bucket_joint_lower_limit}" upper="${gripper_bucket_joint_upper_limit}"/>
         <dynamics damping="${fourbar_joint_damping}" friction="${fourbar_joint_friction}"/>
         <mimic joint="gripper_gear_left_joint" multiplier="-1.0" offset="0.0"/>
@@ -306,5 +315,5 @@
         <axis xyz="0 -1 0"/>
         <limit effort="500" velocity="1.0"
-               lower="${gripper_joint_lower_limit}" upper="${gripper_joint_upper_limit}"/>
+               lower="${gripper_bucket_joint_lower_limit}" upper="${gripper_bucket_joint_upper_limit}"/>
         <dynamics damping="${fourbar_joint_damping}" friction="${fourbar_joint_friction}"/>
         <mimic joint="gripper_gear_left_joint" multiplier="-1.0" offset="0.0"/>

Commit message: commit

File: src/aries/urdf/gripper_camera.xacro (robot description, xacro)
@@ -22,7 +22,14 @@
           /gripper_camera/aligned_depth_to_color/image_raw  (alias of the depth image)
     -->
-    <!-- Mount joint - attaches camera to gripper base -->
+    <!-- Mount joint - attaches camera to gripper base.
+         gripper_camera_y IS SET BY WHOEVER INCLUDES THIS FILE and there is no
+         default on purpose. The bracket is modelled in neither gripper's base
+         mesh, so the offset comes from the camera holes in the mount casting,
+         and the two grippers do not agree: v2 puts them 47.439 mm out in +Y,
+         the ST3215 mount 65.274 mm. A default here would silently hang the
+         camera in the wrong place on whichever gripper did not match it, and a
+         wrong extrinsic is the one error the grasp stack cannot see. -->
     <joint name="gripper_camera_joint" type="fixed">
-        <origin xyz="0.0 0.047439 0.035208" rpy="0 -1.57 -1.57"/>
+        <origin xyz="0.0 ${gripper_camera_y} 0.035208" rpy="0 -1.57 -1.57"/>
         <parent link="arm_gripper_base_link"/>
         <child link="gripper_camera_bottom_screw_frame"/>

File: src/aries/urdf/gripper_v2.xacro (robot description, xacro)
@@ -467,5 +467,9 @@
          pose is unchanged: it hangs off a bracket that is modelled in neither
          base mesh, and the base solid itself is the same part in the same
-         frame, so the old extrinsics still apply. -->
+         frame, so the old extrinsics still apply. The offset moved out of that
+         file when gripper_st3215.xacro arrived, because that mount's camera
+         holes sit 18.2 mm further out; the value here is the one this file
+         always used. -->
+    <xacro:property name="gripper_camera_y" value="0.047439"/>
     <xacro:include filename="gripper_camera.xacro" />
 </robot>

File: src/aries/urdf/igus_rebel2.control.xacro (robot description, xacro)
@@ -2,5 +2,5 @@
 <!-- igus_rebel.control.xacro -->
 <robot xmlns:xacro="http://www.ros.org/wiki/xacro">
-    <xacro:macro name="igus_rebel_control" params="arm_id hardware_protocol arm_hardware_protocol:='' gripper_hardware_protocol:='' serial_port:='/dev/ttyACM0'">
+    <xacro:macro name="igus_rebel_control" params="arm_id hardware_protocol arm_hardware_protocol:='' gripper_hardware_protocol:='' serial_port:='/dev/ttyACM0' gripper_type:='v2' servo_bus_port:='/dev/aries_servo_bus' servo_bus_baud:='1000000' servo_id:='1' gripper_closed_steps:='3000' gripper_servo_invert:='false'">
         <xacro:macro name="joint_control" params="joint">
             <joint name="${joint}">
@@ -71,24 +71,40 @@
                      stay so the followers still report their measured
                      positions. -->
-                <joint name="gripper_gear_right_joint">
-                    <state_interface name="position" />
-                    <state_interface name="velocity" />
-                </joint>
-                <joint name="gripper_link_left_joint">
-                    <state_interface name="position" />
-                    <state_interface name="velocity" />
-                </joint>
-                <joint name="gripper_link_right_joint">
-                    <state_interface name="position" />
-                    <state_interface name="velocity" />
-                </joint>
-                <joint name="gripper_bucket_left_joint">
-                    <state_interface name="position" />
-                    <state_interface name="velocity" />
-                </joint>
-                <joint name="gripper_bucket_right_joint">
-                    <state_interface name="position" />
-                    <state_interface name="velocity" />
-                </joint>
+                <xacro:if value="${gripper_type == 'v2'}">
+                    <joint name="gripper_gear_right_joint">
+                        <state_interface name="position" />
+                        <state_interface name="velocity" />
+                    </joint>
+                    <joint name="gripper_link_left_joint">
+                        <state_interface name="position" />
+                        <state_interface name="velocity" />
+                    </joint>
+                    <joint name="gripper_link_right_joint">
+                        <state_interface name="position" />
+                        <state_interface name="velocity" />
+                    </joint>
+                    <joint name="gripper_bucket_left_joint">
+                        <state_interface name="position" />
+                        <state_interface name="velocity" />
+                    </joint>
+                    <joint name="gripper_bucket_right_joint">
+                        <state_interface name="position" />
+                        <state_interface name="velocity" />
+                    </joint>
+                </xacro:if>
+                <!-- The ST3215 gripper has two followers, not five, and they
+                     are PRISMATIC: their state is metres, not radians. Its
+                     fingertips are bolted to the racks with fixed joints, so
+                     there is nothing else to report. -->
+                <xacro:if value="${gripper_type == 'st3215'}">
+                    <joint name="gripper_rack_left_joint">
+                        <state_interface name="position" />
+                        <state_interface name="velocity" />
+                    </joint>
+                    <joint name="gripper_rack_right_joint">
+                        <state_interface name="position" />
+                        <state_interface name="velocity" />
+                    </joint>
+                </xacro:if>
             </xacro:if>
         </ros2_control>
@@ -98,11 +114,17 @@
                     <plugin>mock_components/GenericSystem</plugin>
                 </hardware>
+                <!-- The command range is the FITTED gripper's, not a shared
+                     constant: v2 stops at -1.57 and the ST3215 runs to -4.065.
+                     Clamping the ST3215 at -1.57 would quietly cap mock runs
+                     at a 32.9 mm jaw gap against the real 82.9. -->
+                <xacro:property name="gripper_mock_min"
+                                value="${-4.065 if gripper_type == 'st3215' else -1.57}"/>
                 <joint name="gripper_gear_left_joint">
                     <command_interface name="position">
-                        <param name="min">-1.57</param>
+                        <param name="min">${gripper_mock_min}</param>
                         <param name="max">0.07</param>
                     </command_interface>
                     <state_interface name="position">
-                        <param name="initial_value">-1.57</param>
+                        <param name="initial_value">${gripper_mock_min}</param>
                     </state_interface>
                     <state_interface name="velocity" />
@@ -126,4 +148,48 @@
             </ros2_control>
         </xacro:if>
+        <!-- The ST3215 gripper does NOT go through the Teensy. Its servo hangs
+             off the rover PC's own USB bus-servo adapter, so this component
+             opens the serial port itself and speaks Feetech STS to it. That is
+             also why it is a separate protocol value rather than another
+             gripper_type branch inside 'rebel': the two grippers reach their
+             servos over different wires, and 'rebel' means "through the
+             Teensy". -->
+        <xacro:if value="${gripper_hardware_protocol == 'st3215'}">
+            <ros2_control name="${arm_id}_gripper" type="system">
+                <hardware>
+                    <plugin>st3215_gripper_hardware/ST3215GripperSystem</plugin>
+                    <param name="port">${servo_bus_port}</param>
+                    <param name="baud">${servo_bus_baud}</param>
+                    <param name="servo_id">${servo_id}</param>
+                    <!-- Servo step at the CLOSED end of travel (q = +0.07), and
+                         the direction a rising step count moves the joint.
+                         The only two numbers here that are NOT derived from the
+                         CAD: they depend on how the pinion was clocked onto the
+                         horn at assembly, so they change whenever the servo is
+                         unbolted. Passed in as launch args - see the package
+                         header for how to measure them. -->
+                    <param name="closed_steps">${gripper_closed_steps}</param>
+                    <param name="invert">${gripper_servo_invert}</param>
+                    <param name="min_pos">-4.065</param>
+                    <param name="max_pos">0.07</param>
+                    <!-- 0 leaves the servo's stored acceleration alone. Do not
+                         set this casually: on this servo the acceleration
+                         register silently caps top speed AND is what produced
+                         a 44 deg overshoot on the bench. -->
+                    <param name="accel">0</param>
+                    <param name="goal_speed">2000</param>
+                    <param name="torque_limit">800</param>
+                </hardware>
+                <joint name="gripper_gear_left_joint">
+                    <command_interface name="position" />
+                    <state_interface name="position" />
+                    <state_interface name="velocity" />
+                    <!-- Real feedback, unlike the Teensy gripper: the ST3215
+                         reports present position, speed and load, so effort
+                         here is a measurement and not an echo. -->
+                    <state_interface name="effort" />
+                </joint>
+            </ros2_control>
+        </xacro:if>
         <xacro:if value="${arm_hardware_protocol == 'gazebo' or (arm_hardware_protocol == '' and hardware_protocol == 'gazebo')}">
             <gazebo>

File: src/aries/urdf/my_robot.urdf.xacro (robot description, xacro)
@@ -1,12 +1,21 @@
 <?xml version="1.0"?>
 <robot xmlns:xacro="http://www.ros.org/wiki/xacro" name="aries">
-  <!-- The REBEL-6DOF-04 gripper (meshing sector gears) is the only gripper
-       this robot is built with. The 85.563 mm four-bar ('new') and the
-       original ('old') are retired to urdf/legacy/ and are not reachable from
-       here; nothing in the fleet runs them any more.
-       The argument is still declared because a dozen launch files pass
-       gripper_type:=v2 down to this file, and an undeclared arg is a hard
-       error. It is accepted and ignored - there is no branch left to take. -->
+  <!-- Which gripper is bolted to the ReBeL tool flange.
+         v2      REBEL-6DOF-04, meshing sector gears on a four-bar, servo
+                 driven through the Teensy. The primary gripper.
+         st3215  rack and pinion, one Waveshare/Feetech ST3215 bus servo wired
+                 straight to the rover PC. The secondary gripper.
+       They are MUTUALLY EXCLUSIVE - both bolt to the same six-hole flange, so
+       only one can be fitted - and swapping between them needs no change
+       anywhere else: both publish the same driver joint name
+       (gripper_gear_left_joint), the same +0.07-closed / negative-open sign
+       convention, the same gripper_bucket_*_link jaw names and the same
+       gripper_tcp at 0.15 m.
+       The 85.563 mm four-bar ('new') and the original ('old') are retired to
+       urdf/legacy/ and are not reachable from here.
+       finger_type applies to v2 only. The ST3215 gripper has one CAD'd pair of
+       scoops and no fingertip interface to swap. -->
   <xacro:arg name="gripper_type" default="v2"/>
+  <xacro:property name="gripper_type" value="$(arg gripper_type)"/>
   <!-- Swappable fingertip - 'bucket', 'maintenance', or 'probe' -->
   <xacro:arg name="finger_type" default="probe"/>
@@ -23,4 +32,27 @@
   <xacro:arg name="serial_port" default="/dev/ttyACM0"/>
   <xacro:property name="serial_port" value="$(arg serial_port)"/>
+  <!-- ST3215 bus-servo adapter, used only by gripper_type:=st3215. The
+       defaults mirror aries_common/config/devices.yaml's servo_bus block; the
+       launch files pass the resolved values in rather than relying on them. -->
+  <xacro:arg name="servo_bus_port" default="/dev/aries_servo_bus"/>
+  <xacro:property name="servo_bus_port" value="$(arg servo_bus_port)"/>
+  <xacro:arg name="servo_bus_baud" default="1000000"/>
+  <xacro:property name="servo_bus_baud" value="$(arg servo_bus_baud)"/>
+  <xacro:arg name="servo_id" default="1"/>
+  <xacro:property name="servo_id" value="$(arg servo_id)"/>
+  <!-- BENCH CALIBRATION for gripper_type:=st3215, and the only two numbers in
+       the whole gripper that cannot be derived from the CAD.
+       gripper_closed_steps  the servo's raw encoder step at q = +0.07 rad,
+                             jaws touching. Depends on how the pinion was
+                             clocked onto the horn at assembly, so it changes
+                             whenever the servo is unbolted.
+       gripper_servo_invert  whether a rising step count closes or opens.
+       They are launch args rather than devices.yaml entries because they are
+       calibration, not device identity - devices.yaml says so in its header.
+       See st3215_gripper_hardware's package header for how to measure them. -->
+  <xacro:arg name="gripper_closed_steps" default="3000"/>
+  <xacro:property name="gripper_closed_steps" value="$(arg gripper_closed_steps)"/>
+  <xacro:arg name="gripper_servo_invert" default="false"/>
+  <xacro:property name="gripper_servo_invert" value="$(arg gripper_servo_invert)"/>
   <xacro:include filename="common_properties.xacro"/>
   <xacro:include filename="aries_gazebo.xacro"/>
@@ -37,5 +69,17 @@
   <xacro:include filename="igus_rebel2.control.xacro"/>
   <!-- Instantiate the arm control macro -->
-  <xacro:igus_rebel_control arm_id="aries" hardware_protocol="${hardware_protocol}" arm_hardware_protocol="${arm_hardware_protocol}" gripper_hardware_protocol="${gripper_hardware_protocol}" serial_port="${serial_port}"/>
-  <xacro:include filename="gripper_v2.xacro"/>
+  <xacro:igus_rebel_control arm_id="aries" hardware_protocol="${hardware_protocol}" arm_hardware_protocol="${arm_hardware_protocol}" gripper_hardware_protocol="${gripper_hardware_protocol}" serial_port="${serial_port}" gripper_type="${gripper_type}" servo_bus_port="${servo_bus_port}" servo_bus_baud="${servo_bus_baud}" servo_id="${servo_id}" gripper_closed_steps="${gripper_closed_steps}" gripper_servo_invert="${gripper_servo_invert}"/>
+  <!-- An unknown gripper_type must fail loudly. Without this the include below
+       simply does not fire and the arm comes up with no end effector at all,
+       which reads in RViz as "the gripper meshes did not load" and sends you
+       looking at mesh paths. -->
+  <xacro:if value="${gripper_type not in ('v2', 'st3215')}">
+    <xacro:gripper_type_must_be_v2_or_st3215/>
+  </xacro:if>
+  <xacro:if value="${gripper_type == 'v2'}">
+    <xacro:include filename="gripper_v2.xacro"/>
+  </xacro:if>
+  <xacro:if value="${gripper_type == 'st3215'}">
+    <xacro:include filename="gripper_st3215.xacro"/>
+  </xacro:if>
 </robot>
