Commit message: commit

File: src/aries/urdf/igus_rebel2.control.xacro (robot description, xacro)
@@ -71,40 +71,27 @@
                      stay so the followers still report their measured
                      positions. -->
-                <xacro:if value="${gripper_type == 'v2'}">
-                    <joint name="gripper_gear_right_joint">
-                        <state_interface name="position" />
-                        <state_interface name="velocity" />
-                    </joint>
-                    <joint name="gripper_link_left_joint">
-                        <state_interface name="position" />
-                        <state_interface name="velocity" />
-                    </joint>
-                    <joint name="gripper_link_right_joint">
-                        <state_interface name="position" />
-                        <state_interface name="velocity" />
-                    </joint>
-                    <joint name="gripper_bucket_left_joint">
-                        <state_interface name="position" />
-                        <state_interface name="velocity" />
-                    </joint>
-                    <joint name="gripper_bucket_right_joint">
-                        <state_interface name="position" />
-                        <state_interface name="velocity" />
-                    </joint>
-                </xacro:if>
-                <!-- The ST3215 gripper has two followers, not five, and they
-                     are PRISMATIC: their state is metres, not radians. Its
-                     fingertips are bolted to the racks with fixed joints, so
-                     there is nothing else to report. -->
-                <xacro:if value="${gripper_type == 'st3215'}">
-                    <joint name="gripper_rack_left_joint">
-                        <state_interface name="position" />
-                        <state_interface name="velocity" />
-                    </joint>
-                    <joint name="gripper_rack_right_joint">
-                        <state_interface name="position" />
-                        <state_interface name="velocity" />
-                    </joint>
-                </xacro:if>
+                <!-- The rack followers are READ ONLY here, and they are
+                     PRISMATIC: their state is metres, not radians.
+                     They used to carry mimic/multiplier params as well, which
+                     coupled them a SECOND time: sdformat converts the URDF
+                     <mimic> tags into real SDF <mimic> constraints (confirmed
+                     with `gz sdf -p`), so DART already enforces the relation
+                     inside the solver. Adding the ros2_control mimic on top
+                     makes gz_ros2_control write a velocity command to the same
+                     joints every cycle, so each DOF carries a hard kinematic
+                     constraint and an independent servo command that know
+                     nothing about each other. Two solvers arguing over one DOF
+                     is what tears a linkage apart on screen while every joint
+                     is individually "satisfied".
+                     The fingertips are bolted to the racks with fixed joints,
+                     so there is nothing else to report. -->
+                <joint name="gripper_rack_left_joint">
+                    <state_interface name="position" />
+                    <state_interface name="velocity" />
+                </joint>
+                <joint name="gripper_rack_right_joint">
+                    <state_interface name="position" />
+                    <state_interface name="velocity" />
+                </joint>
             </xacro:if>
         </ros2_control>
@@ -114,10 +101,9 @@
                     <plugin>mock_components/GenericSystem</plugin>
                 </hardware>
-                <!-- The command range is the FITTED gripper's, not a shared
-                     constant: v2 stops at -1.57 and the ST3215 runs to -4.065.
-                     Clamping the ST3215 at -1.57 would quietly cap mock runs
-                     at a 32.9 mm jaw gap against the real 82.9. -->
+                <!-- The command range is derived from the calibration YAML,
+                     the same value the real backend clamps to, so a mock run
+                     covers the same jaw gap as the hardware. -->
                 <xacro:property name="gripper_mock_min"
-                                value="${gripper_command_open if gripper_type == 'st3215' else -1.57}"/>
+                                value="${gripper_command_open}"/>
                 <joint name="gripper_gear_left_joint">
                     <command_interface name="position">
@@ -132,27 +118,17 @@
             </ros2_control>
         </xacro:if>
-        <xacro:if value="${gripper_hardware_protocol == 'rebel' or (gripper_hardware_protocol == '' and hardware_protocol == 'rebel')}">
-            <ros2_control name="${arm_id}_gripper" type="system">
-                <hardware>
-                    <plugin>teensy_gripper_hardware/TeensyGripperSystem</plugin>
-                    <param name="cmd_topic">/gripper/cmd</param>
-                    <param name="state_topic">/gripper/state</param>
-                    <param name="min_pos">-1.57</param>
-                    <param name="max_pos">0.07</param>
-                </hardware>
-                <joint name="gripper_gear_left_joint">
-                    <command_interface name="position" />
-                    <state_interface name="position" />
-                    <state_interface name="velocity" />
-                </joint>
-            </ros2_control>
-        </xacro:if>
-        <!-- The ST3215 gripper does NOT go through the Teensy. Its servo hangs
-             off the rover PC's own USB bus-servo adapter, so this component
-             opens the serial port itself and speaks Feetech STS to it. That is
-             also why it is a separate protocol value rather than another
-             gripper_type branch inside 'rebel': the two grippers reach their
-             servos over different wires, and 'rebel' means "through the
-             Teensy". -->
+        <!-- THERE IS NO TEENSY GRIPPER BACKEND ANY MORE. gripper_v2 and its
+             teensy_gripper_hardware plugin are retired (urdf/legacy/, and the
+             package carries a COLCON_IGNORE).
+             THE TEENSY ITSELF IS VERY MUCH STILL HERE, running the drill, the
+             stack light and the load cells over one micro-ROS link. Do not read
+             the absence of a gripper block here as the board being gone - the
+             agent that serves it is started by the launch whenever the board is
+             present, independent of the gripper.
+             The ST3215's servo hangs off the rover PC's own USB bus-servo
+             adapter instead, so the component below opens the serial port
+             itself and speaks Feetech STS to it. That is why it is its own
+             gripper_hardware_protocol value: the wire is different, not just
+             the plugin. -->
         <xacro:if value="${gripper_hardware_protocol == 'st3215'}">
             <ros2_control name="${arm_id}_gripper" type="system">

File: src/aries/urdf/my_robot.urdf.xacro (robot description, xacro)
@@ -1,20 +1,16 @@
 <?xml version="1.0"?>
 <robot xmlns:xacro="http://www.ros.org/wiki/xacro" name="aries">
-  <!-- Which gripper is bolted to the ReBeL tool flange.
-         v2      REBEL-6DOF-04, meshing sector gears on a four-bar, servo
-                 driven through the Teensy. The primary gripper.
-         st3215  rack and pinion, one Waveshare/Feetech ST3215 bus servo wired
-                 straight to the rover PC. The secondary gripper.
-       They are MUTUALLY EXCLUSIVE - both bolt to the same six-hole flange, so
-       only one can be fitted - and swapping between them needs no change
-       anywhere else: both publish the same driver joint name
-       (gripper_gear_left_joint), the same +0.07-closed / negative-open sign
-       convention, the same gripper_bucket_*_link jaw names and the same
-       gripper_tcp at 0.15 m.
-       The 85.563 mm four-bar ('new') and the original ('old') are retired to
-       urdf/legacy/ and are not reachable from here.
-       finger_type applies to v2 only. The ST3215 gripper has one CAD'd pair of
-       scoops and no fingertip interface to swap. -->
-  <xacro:arg name="gripper_type" default="v2"/>
+  <!-- THE ST3215 RACK-AND-PINION IS THE ONLY GRIPPER as of 2026-08-30.
+       gripper_v2 (the REBEL-6DOF-04 four-bar, servo driven through the Teensy)
+       is retired to urdf/legacy/ and its meshes to meshes/unused/gripper_v2/,
+       alongside the older 'new' and 'old' grippers. Nothing in the fleet runs
+       them.
+       gripper_type is still DECLARED because a dozen launch files pass it down
+       and an undeclared arg is a hard error, but 'st3215' is the only accepted
+       value and every launch file's choices= is narrowed to it. finger_type is
+       likewise accepted and ignored: it selected between v2's three swappable
+       fingertips, and this gripper has one CAD'd pair of scoops with no
+       fingertip interface. -->
+  <xacro:arg name="gripper_type" default="st3215"/>
   <xacro:property name="gripper_type" value="$(arg gripper_type)"/>
   <!-- Swappable fingertip - 'bucket', 'maintenance', or 'probe' -->
@@ -74,16 +70,10 @@
   <!-- Instantiate the arm control macro -->
   <xacro:igus_rebel_control arm_id="aries" hardware_protocol="${hardware_protocol}" arm_hardware_protocol="${arm_hardware_protocol}" gripper_hardware_protocol="${gripper_hardware_protocol}" serial_port="${serial_port}" gripper_type="${gripper_type}" servo_bus_port="${servo_bus_port}" servo_bus_baud="${servo_bus_baud}" servo_id="${servo_id}" gripper_closed_steps="${gripper_closed_steps}" gripper_servo_invert="${gripper_servo_invert}" gripper_command_open="${gripper_command_open}"/>
-  <!-- An unknown gripper_type must fail loudly. Without this the include below
-       simply does not fire and the arm comes up with no end effector at all,
-       which reads in RViz as "the gripper meshes did not load" and sends you
-       looking at mesh paths. -->
-  <xacro:if value="${gripper_type not in ('v2', 'st3215')}">
-    <xacro:gripper_type_must_be_v2_or_st3215/>
+  <!-- A gripper_type this file does not build must fail loudly rather than
+       leave the arm with no end effector, which reads in RViz as "the gripper
+       meshes did not load" and sends you looking at mesh paths. -->
+  <xacro:if value="${gripper_type != 'st3215'}">
+    <xacro:gripper_type_must_be_st3215/>
   </xacro:if>
-  <xacro:if value="${gripper_type == 'v2'}">
-    <xacro:include filename="gripper_v2.xacro"/>
-  </xacro:if>
-  <xacro:if value="${gripper_type == 'st3215'}">
-    <xacro:include filename="gripper_st3215.xacro"/>
-  </xacro:if>
+  <xacro:include filename="gripper_st3215.xacro"/>
 </robot>
