Commit message: commit

File: src/aries/urdf/aries_base.xacro (robot description, xacro)
@@ -63,5 +63,5 @@
                     rpy="0 0 0" />
             <geometry>
-                <mesh filename="${mesh_location}/base_link.STL" />
+                <mesh filename="${mesh_location}/base_link_v2.stl" />
             </geometry>
             <material
@@ -74,5 +74,5 @@
                     rpy="0 0 0" />
             <geometry>
-                <mesh filename="${mesh_location}/base_link.STL" />
+                <mesh filename="${mesh_location}/base_link_v2.stl" />
             </geometry>
         </collision>

Commit message: commit

File: src/aries/urdf/aries_base.xacro (robot description, xacro)
@@ -63,10 +63,6 @@
                     rpy="0 0 0" />
             <geometry>
-                <mesh filename="${mesh_location}/base_link_v2.stl" />
+                <mesh filename="${mesh_location}/base_link_v3.glb" />
             </geometry>
-            <material
-                name="">
-                <color rgba="1 1 1 1" />
-            </material>
         </visual>
         <collision>
@@ -74,5 +70,5 @@
                     rpy="0 0 0" />
             <geometry>
-                <mesh filename="${mesh_location}/base_link_v2.stl" />
+                <mesh filename="${mesh_location}/base_link_v3.stl" />
             </geometry>
         </collision>

File: src/aries/urdf/aries_gazebo.xacro (robot description, xacro)
@@ -3,5 +3,4 @@
   <!-- Gazebo Materials -->
   <gazebo reference="base_link">
-    <material>Gazebo/Gray</material>
     <mu1>0.2</mu1>
     <mu2>0.2</mu2>
@@ -44,5 +43,4 @@
   </gazebo>
   <gazebo reference="L_1_Wheel_Link">
-    <material>Gazebo/Black</material>
     <mu1>1.4</mu1>
     <mu2>0.35</mu2>
@@ -54,5 +52,4 @@
   </gazebo>
   <gazebo reference="L_2_Wheel_Link">
-    <material>Gazebo/Black</material>
     <mu1>1.4</mu1>
     <mu2>0.35</mu2>
@@ -64,5 +61,4 @@
   </gazebo>
   <gazebo reference="L_3_Wheel_Link">
-    <material>Gazebo/Black</material>
     <mu1>1.4</mu1>
     <mu2>0.35</mu2>
@@ -74,5 +70,4 @@
   </gazebo>
   <gazebo reference="R_1_Wheel_Link">
-    <material>Gazebo/Black</material>
     <mu1>1.4</mu1>
     <mu2>0.35</mu2>
@@ -84,5 +79,4 @@
   </gazebo>
   <gazebo reference="R_2_Wheel_Link">
-    <material>Gazebo/Black</material>
     <mu1>1.4</mu1>
     <mu2>0.35</mu2>
@@ -94,5 +88,4 @@
   </gazebo>
   <gazebo reference="R_3_Wheel_Link">
-    <material>Gazebo/Black</material>
     <mu1>1.4</mu1>
     <mu2>0.35</mu2>

File: src/aries/urdf/camera.xacro (robot description, xacro)
@@ -21,6 +21,7 @@
         </visual>
         <collision>
+            <origin xyz="-0.0126 0 0" rpy="0 0 0"/>
             <geometry>
-                <mesh filename="${mesh_location}/d435.stl"/>
+                <box size="0.0252 0.090 0.025"/>
             </geometry>
         </collision>

File: src/aries/urdf/d435i.xacro (robot description, xacro)
@@ -42,6 +42,7 @@
         </visual>
         <collision>
+            <origin xyz="-0.0126 0 0" rpy="0 0 0"/>
             <geometry>
-                <mesh filename="${mesh_location}/d435.stl"/>
+                <box size="0.0252 0.090 0.025"/>
             </geometry>
         </collision>

File: src/aries/urdf/gripper_camera.xacro (robot description, xacro)
@@ -50,6 +50,7 @@
         </visual>
         <collision>
+            <origin xyz="-0.0126 0 0" rpy="0 0 0"/>
             <geometry>
-                <mesh filename="${mesh_location}/d435.stl"/>
+                <box size="0.0252 0.090 0.025"/>
             </geometry>
         </collision>

File: src/aries/urdf/left_link.xacro (robot description, xacro)
@@ -53,12 +53,11 @@
             <origin xyz="0 0 0" rpy="${-PI/2} 0 ${PI}"/>
             <geometry>
-                <mesh filename="${mesh_location}/L_1_Wheel_Link.STL"/>
+                <mesh filename="${mesh_location}/L_1_Wheel_Link_v2.glb"/>
             </geometry>
-            <material name="blue"/>
         </visual>
         <collision>
-            <origin xyz="0 -0.035 0" rpy="${PI/2} 0 0"/>
+            <origin xyz="0 0 0" rpy="${PI/2} 0 0"/>
             <geometry>
-                <cylinder radius="${wheel_radius}" length="${wheel_thickness}"/>
+                <mesh filename="${mesh_location}/L_1_Wheel_Link_v2.stl"/>
             </geometry>
         </collision>
@@ -87,12 +86,11 @@
             <origin xyz="0 0 0" rpy="${-PI/2} 0 ${PI}"/>
             <geometry>
-                <mesh filename="${mesh_location}/L_2_Wheel_Link.STL"/>
+                <mesh filename="${mesh_location}/L_2_Wheel_Link_v2.glb"/>
             </geometry>
-            <material name="blue"/>
         </visual>
         <collision>
-            <origin xyz="0 -0.035 0" rpy="${PI/2} 0 0"/>
+            <origin xyz="0 0 0" rpy="${PI/2} 0 0"/>
             <geometry>
-                <cylinder radius="${wheel_radius}" length="${wheel_thickness}"/>
+                 <mesh filename="${mesh_location}/L_2_Wheel_Link_v2.stl"/>
             </geometry>
         </collision>
@@ -121,12 +119,11 @@
             <origin xyz="0 0 0" rpy="${-PI/2} 0 ${PI}"/>
             <geometry>
-                <mesh filename="${mesh_location}/L_3_Wheel_Link.STL"/>
+                <mesh filename="${mesh_location}/L_3_Wheel_Link_v2.glb"/>
             </geometry>
-            <material name="blue"/>
         </visual>
         <collision>
-            <origin xyz="0 -0.035 0" rpy="${PI/2} 0 0"/>
+            <origin xyz="0 0 0" rpy="${PI/2} 0 0"/>
             <geometry>
-                <cylinder radius="${wheel_radius}" length="${wheel_thickness}"/>
+                <mesh filename="${mesh_location}/L_3_Wheel_Link_v2.stl"/>
             </geometry>
         </collision>

File: src/aries/urdf/right_link.xacro (robot description, xacro)
@@ -56,12 +56,11 @@
             <origin xyz="0 0 0" rpy="${PI/2} 0 ${PI}"/>
             <geometry>
-                <mesh filename="${mesh_location}/R_1_Wheel_Link.STL"/>
+                <mesh filename="${mesh_location}/R_1_Wheel_Link_v2.glb"/>
             </geometry>
-            <material name="blue"/>
         </visual>
         <collision>
-            <origin xyz="0 0.035 0" rpy="${PI/2} 0 0"/>
+            <origin xyz="0 0 0" rpy="${PI/2} 0 0"/>
             <geometry>
-                <cylinder radius="${wheel_radius}" length="${wheel_thickness}"/>
+                <mesh filename="${mesh_location}/R_1_Wheel_Link_v2.stl"/>
             </geometry>
         </collision>
@@ -90,12 +89,11 @@
             <origin xyz="0 0 0" rpy="${PI/2} 0 ${PI}"/>
             <geometry>
-                <mesh filename="${mesh_location}/R_2_Wheel_Link.STL"/>
+                <mesh filename="${mesh_location}/R_2_Wheel_Link_v2.glb"/>
             </geometry>
-            <material name="blue"/>
         </visual>
         <collision>
-            <origin xyz="0 0.035 0" rpy="${PI/2} 0 0"/>
+            <origin xyz="0 0 0" rpy="${PI/2} 0 0"/>
             <geometry>
-                <cylinder radius="${wheel_radius}" length="${wheel_thickness}"/>
+                <mesh filename="${mesh_location}/R_2_Wheel_Link_v2.stl"/>
             </geometry>
         </collision>
@@ -125,12 +123,11 @@
             <origin xyz="0 0 0" rpy="${PI/2} 0 ${PI}"/>
             <geometry>
-                <mesh filename="${mesh_location}/R_3_Wheel_Link.STL"/>
+                <mesh filename="${mesh_location}/R_2_Wheel_Link_v2.glb"/>
             </geometry>
-            <material name="blue"/>
         </visual>
         <collision>
             <origin xyz="0 0.035 0" rpy="${PI/2} 0 0"/>
             <geometry>
-                <cylinder radius="${wheel_radius}" length="${wheel_thickness}"/>
+                <mesh filename="${mesh_location}/R_2_Wheel_Link_v2.stl"/>
             </geometry>
         </collision>

Commit message: commit

File: src/aries/urdf/aries_base.xacro (robot description, xacro)
@@ -43,5 +43,7 @@
         <parent link="base_footprint" />
         <child link="base_link" />
-        <origin xyz="0 0 0.165" rpy="0 0 0" />
+        <!-- See base_link_height in common_properties.xacro. Was 0.165, which
+             sat 41 mm below the real wheel contact plane. -->
+        <origin xyz="0 0 ${base_link_height}" rpy="0 0 0" />
     </joint>
     <!-- Base Link -->

File: src/aries/urdf/common_properties.xacro (robot description, xacro)
@@ -16,4 +16,16 @@
   <xacro:property name="wheel_radius" value="0.1100"/>
   <xacro:property name="wheel_thickness" value="0.070"/>
+  <!-- Height of base_link above the wheel contact plane.
+       base_footprint is by convention the ground projection of the base, so
+       this must place the bottom of the wheels at exactly z = 0. It was
+       hard-coded to 0.165, which left the wheels 41 mm BELOW base_footprint —
+       everything treating that frame as ground (EKF, odom->base_footprint,
+       nav ground filtering, the LiDAR height) inherited that error.
+       Forward kinematics through the rocker/bogie chain puts the front and
+       middle wheel centres 0.0964 m below base_link, so the base must stand
+       one wheel radius above that. Derived rather than hard-coded so the two
+       can no longer drift apart if wheel_radius changes. -->
+  <xacro:property name="wheel_centre_below_base_link" value="0.0964"/>
+  <xacro:property name="base_link_height" value="${wheel_radius + wheel_centre_below_base_link}"/>
   <!-- Mesh locations -->
   <xacro:property name="mesh_location" value="package://aries/meshes"/>

File: src/aries/urdf/gripper_new.xacro (robot description, xacro)
@@ -13,4 +13,22 @@
          same mount pivots, so only the visual/collision mesh changes. -->
     <xacro:property name="finger_mesh" value="gripper_${finger_type}.stl"/>
+    <!-- Axial correction for where the fingertip actually sits on the bar.
+         The modelled tip sat 50 mm short of the real one: measured against
+         hardware with a probe actually gripped, the attached mesh landed
+         50.2 mm up the shaft from the real probe, with only 1.9 mm lateral and
+         1.3 deg of axis error - i.e. the error is purely along the finger, not
+         a pivot or bar-length problem (see attached_probe_axial_offset_m in
+         aries_vision_grasp/config/vision_grasp_params.yaml, which was the
+         workaround for exactly this). The modelled contact point sat at
+         z=0.220 where the real pinch is ~0.270.
+         Consequences of the old value: RViz drew the jaws 50 mm short, so they
+         could be touching a wheel in reality while the model showed clearance,
+         and MoveIt's collision model inherited the same blind spot.
+         Applied to the fingertip mesh only. The four-bar pivots are correct -
+         gripper_bucket_*_joint IS the gear bar's tip, which is what a four-bar
+         pivot means - so nothing about the linkage motion changes. Set to 0 to
+         restore the old geometry. If you measure flange-to-tip on the real
+         gripper (closed), the model should now read 397.2 mm; adjust here. -->
+    <xacro:property name="finger_axial_correction" value="0.0"/>
     <!-- Mass properties computed from each mesh by tetrahedron decomposition at
          1050 kg/m^3 (near-solid printed plastic), COM and inertia taken about
@@ -264,9 +282,9 @@
     <!--gripper_bucket_left Link -->
     <link name="gripper_bucket_left_link">
-        <xacro:gripper_inertial mass="${finger_mass}" cx="0.0" cy="${finger_com_y}" cz="${finger_com_z}"
+        <xacro:gripper_inertial mass="${finger_mass}" cx="0.0" cy="${finger_com_y}" cz="${finger_com_z + finger_axial_correction}"
                                 ixx="${finger_ixx}" iyy="${finger_iyy}" izz="${finger_izz}"
                                 iyz="${finger_iyz}"/>
         <visual>
-            <origin xyz="0 0 0"
+            <origin xyz="0 0 ${finger_axial_correction}"
                     rpy="0 0 0" />
             <geometry>
@@ -279,5 +297,5 @@
         </visual>
         <collision>
-            <origin xyz="0 0 0"
+            <origin xyz="0 0 ${finger_axial_correction}"
                     rpy="0 0 0" />
             <geometry>
@@ -336,9 +354,9 @@
     <!--gripper_bucket_right Link -->
     <link name="gripper_bucket_right_link">
-        <xacro:gripper_inertial mass="${finger_mass}" cx="0.0" cy="${finger_com_y}" cz="${finger_com_z}"
+        <xacro:gripper_inertial mass="${finger_mass}" cx="0.0" cy="${finger_com_y}" cz="${finger_com_z + finger_axial_correction}"
                                 ixx="${finger_ixx}" iyy="${finger_iyy}" izz="${finger_izz}"
                                 iyz="${finger_iyz}"/>
         <visual>
-            <origin xyz="0 0 0"
+            <origin xyz="0 0 ${finger_axial_correction}"
                     rpy="0 0 0" />
             <geometry>
@@ -351,5 +369,5 @@
         </visual>
         <collision>
-            <origin xyz="0 0 0"
+            <origin xyz="0 0 ${finger_axial_correction}"
                     rpy="0 0 0" />
             <geometry>
@@ -400,4 +418,14 @@
     <!-- Visual constraint markers to show four-bar connection -->
     <link name="fourbar_constraint_visual_left">
+        <!-- Pure RViz marker for the four-bar pivot: no collision on purpose,
+             so it can never obstruct planning. It still needs an inertial or
+             MoveIt/KDL warns about the link on every node start; the value is
+             deliberately negligible so it cannot perturb the gripper dynamics
+             (the real finger links are ~0.4 kg). -->
+        <inertial>
+            <origin xyz="0 0 0" rpy="0 0 0"/>
+            <mass value="1e-6"/>
+            <inertia ixx="1e-9" ixy="0" ixz="0" iyy="1e-9" iyz="0" izz="1e-9"/>
+        </inertial>
         <visual>
             <origin xyz="0 0 0" rpy="0 0 0"/>
@@ -422,4 +450,11 @@
     </joint>
     <link name="fourbar_constraint_visual_right">
+        <!-- See fourbar_constraint_visual_left: marker only, negligible
+             inertial purely to keep MoveIt/KDL from warning on every start. -->
+        <inertial>
+            <origin xyz="0 0 0" rpy="0 0 0"/>
+            <mass value="1e-6"/>
+            <inertia ixx="1e-9" ixy="0" ixz="0" iyy="1e-9" iyz="0" izz="1e-9"/>
+        </inertial>
         <visual>
             <origin xyz="0 0 0" rpy="0 0 0"/>

File: src/aries/urdf/right_link.xacro (robot description, xacro)
@@ -189,5 +189,8 @@
         <parent link="R_Rocker_Link" />
         <child link="aux_R_Rocker_Link" />
-        <limit lower="-3.14" upper="3.14" effort="0.0" velocity="5"/>
+        <!-- effort was 0.0 while the mirrored aux_L_Rocker_joint had 50, so
+             this side could exert no torque at all. Everything else about the
+             two joints mirrors exactly, so the zero was a typo. -->
+        <limit lower="-3.14" upper="3.14" effort="50" velocity="5"/>
         <dynamics damping="0.05" friction="0.0"/>
         <axis xyz="0 0 1" />

Commit message: commit

File: src/aries/urdf/aries_base.xacro (robot description, xacro)
@@ -52,12 +52,18 @@
             <origin xyz="-0.0194894545849965 0.000308596526751935 0.119828029892907"
                     rpy="0 0 0" />
-            <mass value="17.5363204791731" />
+            <!-- The complete competition rover weighs 90 kg. The other links
+                 total 49.0157953866879 kg with the default bucket fingertip,
+                 so batteries, electronics and the
+                 remaining chassis hardware are represented here. The inertia
+                 tensor is scaled with mass from the original CAD tensor,
+                 preserving the chassis radii of gyration. -->
+            <mass value="40.9842046133121" />
             <inertia
-                ixx="0.242660790998556"
-                ixy="-9.00009815481889E-05"
-                ixz="0.0234683038167963"
-                iyy="0.514730499629884"
-                iyz="2.70300300277055E-11"
-                izz="0.664242254581203" />
+                ixx="0.567123503572166"
+                ixy="-0.000210341653344592"
+                ixz="0.0548478665577117"
+                iyy="1.20297870597186"
+                iyz="6.31719911069787E-11"
+                izz="1.55240322545973" />
         </inertial>
         <visual>

File: src/aries/urdf/aries_gazebo.xacro (robot description, xacro)
@@ -43,59 +43,83 @@
   </gazebo>
   <gazebo reference="L_1_Wheel_Link">
-    <!-- Lugged tire: dry polymer tread has more grip than the soil can carry.
-         The Mars-yard surface therefore caps longitudinal traction at 0.60;
-         lower lateral grip permits physical scrub during skid steering. -->
-    <mu1>0.85</mu1>
-    <mu2>0.42</mu2>
-    <kp>1000000.0</kp>
-    <kd>100.0</kd>
-    <minDepth>0.001</minDepth>
-    <maxVel>0.1</maxVel>
-    <fdir1>1 0 0</fdir1>
+    <!-- The cylinder-local Z axis is the wheel axle, so fdir1 and mu1 are
+         lateral. mu2 is longitudinal, capped to 0.65 by the yard surface.
+         WheelSlip below adds speed-dependent granular-soil compliance. -->
+    <mu1>0.42</mu1>
+    <mu2>0.85</mu2>
+    <kp>1000000.0</kp>
+    <kd>100.0</kd>
+    <minDepth>0.001</minDepth>
+    <maxVel>0.1</maxVel>
+    <fdir1>0 0 1</fdir1>
   </gazebo>
   <gazebo reference="L_2_Wheel_Link">
-    <mu1>0.85</mu1>
-    <mu2>0.42</mu2>
-    <kp>1000000.0</kp>
-    <kd>100.0</kd>
-    <minDepth>0.001</minDepth>
-    <maxVel>0.1</maxVel>
-    <fdir1>1 0 0</fdir1>
+    <mu1>0.42</mu1>
+    <mu2>0.85</mu2>
+    <kp>1000000.0</kp>
+    <kd>100.0</kd>
+    <minDepth>0.001</minDepth>
+    <maxVel>0.1</maxVel>
+    <fdir1>0 0 1</fdir1>
   </gazebo>
   <gazebo reference="L_3_Wheel_Link">
-    <mu1>0.85</mu1>
-    <mu2>0.42</mu2>
-    <kp>1000000.0</kp>
-    <kd>100.0</kd>
-    <minDepth>0.001</minDepth>
-    <maxVel>0.1</maxVel>
-    <fdir1>1 0 0</fdir1>
+    <mu1>0.42</mu1>
+    <mu2>0.85</mu2>
+    <kp>1000000.0</kp>
+    <kd>100.0</kd>
+    <minDepth>0.001</minDepth>
+    <maxVel>0.1</maxVel>
+    <fdir1>0 0 1</fdir1>
   </gazebo>
   <gazebo reference="R_1_Wheel_Link">
-    <mu1>0.85</mu1>
-    <mu2>0.42</mu2>
-    <kp>1000000.0</kp>
-    <kd>100.0</kd>
-    <minDepth>0.001</minDepth>
-    <maxVel>0.1</maxVel>
-    <fdir1>1 0 0</fdir1>
+    <mu1>0.42</mu1>
+    <mu2>0.85</mu2>
+    <kp>1000000.0</kp>
+    <kd>100.0</kd>
+    <minDepth>0.001</minDepth>
+    <maxVel>0.1</maxVel>
+    <fdir1>0 0 1</fdir1>
   </gazebo>
   <gazebo reference="R_2_Wheel_Link">
-    <mu1>0.85</mu1>
-    <mu2>0.42</mu2>
-    <kp>1000000.0</kp>
-    <kd>100.0</kd>
-    <minDepth>0.001</minDepth>
-    <maxVel>0.1</maxVel>
-    <fdir1>1 0 0</fdir1>
+    <mu1>0.42</mu1>
+    <mu2>0.85</mu2>
+    <kp>1000000.0</kp>
+    <kd>100.0</kd>
+    <minDepth>0.001</minDepth>
+    <maxVel>0.1</maxVel>
+    <fdir1>0 0 1</fdir1>
   </gazebo>
   <gazebo reference="R_3_Wheel_Link">
-    <mu1>0.85</mu1>
-    <mu2>0.42</mu2>
-    <kp>1000000.0</kp>
-    <kd>100.0</kd>
-    <minDepth>0.001</minDepth>
-    <maxVel>0.1</maxVel>
-    <fdir1>1 0 0</fdir1>
+    <mu1>0.42</mu1>
+    <mu2>0.85</mu2>
+    <kp>1000000.0</kp>
+    <kd>100.0</kd>
+    <minDepth>0.001</minDepth>
+    <maxVel>0.1</maxVel>
+    <fdir1>0 0 1</fdir1>
+  </gazebo>
+  <!-- Gazebo's supported deformable-terrain approximation. The 90 kg rover
+       has an average static wheel load of 90 * 9.8 / 6 = 147 N. Compliance
+       gives about 13% longitudinal and 15% lateral slip at the respective
+       friction limits instead of the perfect no-slip behaviour of Coulomb
+       contact alone. -->
+  <gazebo>
+    <plugin filename="gz-sim-wheel-slip-system"
+            name="gz::sim::systems::WheelSlip">
+      <xacro:macro name="marsyard_wheel_slip" params="link_name">
+        <wheel link_name="${link_name}">
+          <slip_compliance_lateral>0.35</slip_compliance_lateral>
+          <slip_compliance_longitudinal>0.20</slip_compliance_longitudinal>
+          <wheel_normal_force>147.0</wheel_normal_force>
+          <wheel_radius>${wheel_radius}</wheel_radius>
+        </wheel>
+      </xacro:macro>
+      <xacro:marsyard_wheel_slip link_name="L_1_Wheel_Link"/>
+      <xacro:marsyard_wheel_slip link_name="L_2_Wheel_Link"/>
+      <xacro:marsyard_wheel_slip link_name="L_3_Wheel_Link"/>
+      <xacro:marsyard_wheel_slip link_name="R_1_Wheel_Link"/>
+      <xacro:marsyard_wheel_slip link_name="R_2_Wheel_Link"/>
+      <xacro:marsyard_wheel_slip link_name="R_3_Wheel_Link"/>
+    </plugin>
   </gazebo>
   <!-- Gazebo Plugin for Joint State Publisher -->

Commit message: commit

File: src/aries/urdf/aries_base.xacro (robot description, xacro)
@@ -35,5 +35,11 @@
         <parent link="base_link"/>
         <child link="imu_frame"/>
-        <origin xyz="0.0 0.0 0.08" rpy="0.0 0.0 0.0"/>
+        <!-- On the top deck, behind the front D435i. The deck plate in
+             base_link_v3.stl is the large up-facing surface at z = 0.212, so
+             0.222 puts the sensor body 10 mm above it; the camera mount post
+             occupies x ~ 0.24, and the camera itself sits at x = 0.2756
+             (d435i.xacro), so x = 0.18 clears both on open deck. Was
+             0 0 0.08, which was buried mid-chassis. -->
+        <origin xyz="0.19 0.06 0.222" rpy="0.0 0.0 0.0"/>
     </joint>
     <!-- Base Footprint - root link for mobile robot (odom frame provided by odometry, not URDF) -->

Commit message: commit

File: src/aries/urdf/aries_base.xacro (robot description, xacro)
@@ -40,6 +40,15 @@
              occupies x ~ 0.24, and the camera itself sits at x = 0.2756
              (d435i.xacro), so x = 0.18 clears both on open deck. Was
-             0 0 0.08, which was buried mid-chassis. -->
-        <origin xyz="0.19 0.06 0.222" rpy="0.0 0.0 0.0"/>
+             0 0 0.08, which was buried mid-chassis.
+             Yaw is pi because the 3DM-GX5-AHRS is bolted into its cradle with
+             the printed X arrow (and the connector it points at) facing the
+             rover's REAR, so device X = -base_link X and device Y = -base_link Y.
+             Roll stays 0 even though the printed triad shows Z into the
+             mounting plate: microstrain.yaml sets use_enu_frame: true, so the
+             driver has already rolled the native NED device frame 180 deg into
+             ENU before publishing. This link describes the frame the driver
+             publishes in (X fwd, Y left, Z up), not the silkscreen; adding that
+             flip here would apply it twice and invert roll and yaw sign. -->
+        <origin xyz="0.19 0.06 0.222" rpy="0.0 0.0 ${pi}"/>
     </joint>
     <!-- Base Footprint - root link for mobile robot (odom frame provided by odometry, not URDF) -->
