Commit message: commit

File: src/aries/urdf/aries_base.xacro (robot description, xacro)
@@ -36,5 +36,5 @@
         <child link="imu_frame"/>
         <!-- On the top deck, behind the front D435i. The deck plate in
-             base_link_v3.stl is the large up-facing surface at z = 0.212, so
+             base.stl is the large up-facing surface at z = 0.212, so
              0.222 puts the sensor body 10 mm above it; the camera mount post
              occupies x ~ 0.24, and the camera itself sits at x = 0.2756
@@ -86,5 +86,5 @@
                     rpy="0 0 0" />
             <geometry>
-                <mesh filename="${mesh_location}/base_link_v3.glb" />
+                <mesh filename="${mesh_location}/base.glb" />
             </geometry>
         </visual>
@@ -93,5 +93,5 @@
                     rpy="0 0 0" />
             <geometry>
-                <mesh filename="${mesh_location}/base_link_v3.stl" />
+                <mesh filename="${mesh_location}/base.stl" />
             </geometry>
         </collision>

File: src/aries/urdf/aries_gazebo.xacro (robot description, xacro)
@@ -3,4 +3,10 @@
   <!-- Gazebo Materials -->
   <gazebo reference="base_link">
+    <mu1>0.2</mu1>
+    <mu2>0.2</mu2>
+    <kp>1000000.0</kp>
+    <kd>100.0</kd>
+  </gazebo>
+  <gazebo reference="drill_link">
     <mu1>0.2</mu1>
     <mu2>0.2</mu2>

File: src/aries/urdf/gripper_v2.xacro (robot description, xacro)
@@ -96,5 +96,19 @@
          export placed on both jaws, which is only valid because each of those
          solids is symmetric about its own mid-plane (the build script asserts
-         it). -->
+         it).
+         The bucket pair is now the 2026-08-19 CAD re-export (new_mesh/
+         gripper_bucket.stl = LEFT, gripper_bucket_2.stl = RIGHT; the handedness
+         is readable off the tip, the left lip stays 50 mm wide to the end while
+         the right narrows to 29 mm so the two nest when closed). That export
+         carries its own datum, so it was re-expressed in these link frames by
+         matching the mount shank - the 15 x 11 mm prism between the base face
+         and the scoop - rather than by bounding box: the resulting solid sits
+         within 0.14 mm mean / 0.29 mm p95 of the mesh
+         build_gripper_v2_meshes.py cuts out of the assembly GLB, so it is the
+         same fingertip, only tessellated finer across the bowl's back wall
+         (the one 3 mm outlier is chord error on that curve). Re-running that
+         script REGENERATES these two files from the GLB and would undo the
+         swap; the numbers below move by under 1.5 mm / 4% if it does, so
+         nothing breaks, but the meshes stop being the CAD-current ones. -->
     <xacro:property name="finger_mesh_left" value="gripper_${finger_type}_left.stl"/>
     <xacro:property name="finger_mesh_right" value="gripper_${finger_type}_right.stl"/>
@@ -106,17 +120,17 @@
          458 g with the bucket fitted, of which 90 g is the servo. -->
     <xacro:property name="finger_mass"
-                    value="${0.0277 if finger_type == 'probe' else (0.0433 if finger_type == 'bucket' else 0.0187)}"/>
+                    value="${0.0277 if finger_type == 'probe' else (0.0417 if finger_type == 'bucket' else 0.0187)}"/>
     <xacro:property name="finger_com_x"
-                    value="${0.01892 if finger_type == 'probe' else (0.00840 if finger_type == 'bucket' else 0.01748)}"/>
+                    value="${0.01892 if finger_type == 'probe' else (0.00745 if finger_type == 'bucket' else 0.01748)}"/>
     <xacro:property name="finger_com_z"
-                    value="${0.05805 if finger_type == 'probe' else (0.05452 if finger_type == 'bucket' else 0.04608)}"/>
+                    value="${0.05805 if finger_type == 'probe' else (0.05483 if finger_type == 'bucket' else 0.04608)}"/>
     <xacro:property name="finger_ixx"
-                    value="${2.343e-05 if finger_type == 'probe' else (3.617e-05 if finger_type == 'bucket' else 1.338e-05)}"/>
+                    value="${2.343e-05 if finger_type == 'probe' else (3.531e-05 if finger_type == 'bucket' else 1.338e-05)}"/>
     <xacro:property name="finger_iyy"
-                    value="${2.362e-05 if finger_type == 'probe' else (3.212e-05 if finger_type == 'bucket' else 1.468e-05)}"/>
+                    value="${2.362e-05 if finger_type == 'probe' else (3.110e-05 if finger_type == 'bucket' else 1.468e-05)}"/>
     <xacro:property name="finger_izz"
-                    value="${3.462e-06 if finger_type == 'probe' else (1.736e-05 if finger_type == 'bucket' else 1.999e-06)}"/>
+                    value="${3.462e-06 if finger_type == 'probe' else (1.619e-05 if finger_type == 'bucket' else 1.999e-06)}"/>
     <xacro:property name="finger_ixz"
-                    value="${-5.067e-06 if finger_type == 'probe' else (6.137e-07 if finger_type == 'bucket' else -4.098e-06)}"/>
+                    value="${-5.067e-06 if finger_type == 'probe' else (4.309e-07 if finger_type == 'bucket' else -4.098e-06)}"/>
     <!-- Reusable inertial block. -->
     <xacro:macro name="gripper_inertial" params="mass cx cy cz ixx iyy izz ixy:=0 ixz:=0 iyz:=0">
@@ -167,39 +181,39 @@
          The visual stays the real mesh. -->
     <xacro:property name="finger_col0_sx"
-                    value="${0.0262 if finger_type == 'probe' else (0.0270 if finger_type == 'bucket' else 0.0261)}"/>
+                    value="${0.0262 if finger_type == 'probe' else (0.0269 if finger_type == 'bucket' else 0.0261)}"/>
     <xacro:property name="finger_col0_sy"
-                    value="${0.0150 if finger_type == 'probe' else (0.0150 if finger_type == 'bucket' else 0.0150)}"/>
+                    value="${0.0150 if finger_type == 'probe' else (0.0151 if finger_type == 'bucket' else 0.0150)}"/>
     <xacro:property name="finger_col0_sz"
-                    value="${0.0335 if finger_type == 'probe' else (0.0368 if finger_type == 'bucket' else 0.0331)}"/>
+                    value="${0.0335 if finger_type == 'probe' else (0.0369 if finger_type == 'bucket' else 0.0331)}"/>
     <xacro:property name="finger_col0_x"
-                    value="${0.00812 if finger_type == 'probe' else (0.00849 if finger_type == 'bucket' else 0.00803)}"/>
+                    value="${0.00812 if finger_type == 'probe' else (0.00847 if finger_type == 'bucket' else 0.00803)}"/>
     <xacro:property name="finger_col0_y"
-                    value="${0.0 if finger_type == 'probe' else (-0.00005 if finger_type == 'bucket' else 0.0)}"/>
+                    value="${0.0 if finger_type == 'probe' else (0.00001 if finger_type == 'bucket' else 0.0)}"/>
     <xacro:property name="finger_col0_z"
                     value="${0.01180 if finger_type == 'probe' else (0.01346 if finger_type == 'bucket' else 0.01165)}"/>
     <xacro:property name="finger_col1_sx"
-                    value="${0.0173 if finger_type == 'probe' else (0.0466 if finger_type == 'bucket' else 0.0174)}"/>
+                    value="${0.0173 if finger_type == 'probe' else (0.0452 if finger_type == 'bucket' else 0.0174)}"/>
     <xacro:property name="finger_col1_sy"
-                    value="${0.0300 if finger_type == 'probe' else (0.0500 if finger_type == 'bucket' else 0.0150)}"/>
+                    value="${0.0300 if finger_type == 'probe' else (0.0502 if finger_type == 'bucket' else 0.0150)}"/>
     <xacro:property name="finger_col1_sz"
-                    value="${0.0335 if finger_type == 'probe' else (0.0368 if finger_type == 'bucket' else 0.0331)}"/>
+                    value="${0.0335 if finger_type == 'probe' else (0.0369 if finger_type == 'bucket' else 0.0331)}"/>
     <xacro:property name="finger_col1_x"
-                    value="${0.01627 if finger_type == 'probe' else (0.00633 if finger_type == 'bucket' else 0.01588)}"/>
+                    value="${0.01627 if finger_type == 'probe' else (0.00537 if finger_type == 'bucket' else 0.01588)}"/>
     <xacro:property name="finger_col1_y"
-                    value="${0.0 if finger_type == 'probe' else (-0.00005 if finger_type == 'bucket' else 0.0)}"/>
+                    value="${0.0 if finger_type == 'probe' else (-0.00009 if finger_type == 'bucket' else 0.0)}"/>
     <xacro:property name="finger_col1_z"
-                    value="${0.04525 if finger_type == 'probe' else (0.05023 if finger_type == 'bucket' else 0.04479)}"/>
+                    value="${0.04525 if finger_type == 'probe' else (0.05033 if finger_type == 'bucket' else 0.04479)}"/>
     <xacro:property name="finger_col2_sx"
                     value="${0.0217 if finger_type == 'probe' else (0.0483 if finger_type == 'bucket' else 0.0216)}"/>
     <xacro:property name="finger_col2_sy"
-                    value="${0.0300 if finger_type == 'probe' else (0.0500 if finger_type == 'bucket' else 0.0150)}"/>
+                    value="${0.0300 if finger_type == 'probe' else (0.0502 if finger_type == 'bucket' else 0.0150)}"/>
     <xacro:property name="finger_col2_sz"
-                    value="${0.0335 if finger_type == 'probe' else (0.0368 if finger_type == 'bucket' else 0.0331)}"/>
+                    value="${0.0335 if finger_type == 'probe' else (0.0369 if finger_type == 'bucket' else 0.0331)}"/>
     <xacro:property name="finger_col2_x"
-                    value="${0.02568 if finger_type == 'probe' else (0.00883 if finger_type == 'bucket' else 0.02522)}"/>
+                    value="${0.02568 if finger_type == 'probe' else (0.00857 if finger_type == 'bucket' else 0.02522)}"/>
     <xacro:property name="finger_col2_y"
-                    value="${0.0 if finger_type == 'probe' else (-0.00005 if finger_type == 'bucket' else 0.0)}"/>
+                    value="${0.0 if finger_type == 'probe' else (-0.00013 if finger_type == 'bucket' else 0.0)}"/>
     <xacro:property name="finger_col2_z"
-                    value="${0.07870 if finger_type == 'probe' else (0.08699 if finger_type == 'bucket' else 0.07793)}"/>
+                    value="${0.07870 if finger_type == 'probe' else (0.08721 if finger_type == 'bucket' else 0.07793)}"/>
     <!-- The bucket's upper two bands are its scoop, and a box fills the bowl:
          the proxy is SOLID where the real tip is a shell. Nothing in these

File: src/aries/urdf/legacy/gripper.xacro (robot description, xacro)
@@ -23,5 +23,5 @@
                     rpy="0 0 0" />
             <geometry>
-                <mesh filename="file://$(find aries)/meshes/gripper_base.stl" />
+                <mesh filename="file://$(find aries)/meshes/unused/gripper_base.stl" />
             </geometry>
             <material
@@ -34,5 +34,5 @@
                     rpy="0 0 0" />
             <geometry>
-                <mesh filename="file://$(find aries)/meshes/gripper_base.stl" />
+                <mesh filename="file://$(find aries)/meshes/unused/gripper_base.stl" />
             </geometry>
         </collision>
@@ -55,5 +55,5 @@
                     rpy="0 0 0" />
             <geometry>
-                <mesh filename="file://$(find aries)/meshes/gripper_left.stl" />
+                <mesh filename="file://$(find aries)/meshes/unused/gripper_left.stl" />
             </geometry>
             <material
@@ -66,5 +66,5 @@
                     rpy="0 0 0" />
             <geometry>
-                <mesh filename="file://$(find aries)/meshes/gripper_left.stl" />
+                <mesh filename="file://$(find aries)/meshes/unused/gripper_left.stl" />
             </geometry>
         </collision>
@@ -95,5 +95,5 @@
                     rpy="0 0 0" />
             <geometry>
-                <mesh filename="file://$(find aries)/meshes/gripper_right.stl" />
+                <mesh filename="file://$(find aries)/meshes/unused/gripper_right.stl" />
             </geometry>
             <material
@@ -106,5 +106,5 @@
                     rpy="0 0 0" />
             <geometry>
-                <mesh filename="file://$(find aries)/meshes/gripper_right.stl" />
+                <mesh filename="file://$(find aries)/meshes/unused/gripper_right.stl" />
             </geometry>
         </collision>
@@ -120,4 +120,4 @@
     </joint>
     <!-- Gripper Camera (D435i) — defined in gripper_camera.xacro -->
-    <xacro:include filename="gripper_camera.xacro" />
+    <xacro:include filename="$(find aries)/urdf/gripper_camera.xacro" />
 </robot>

File: src/aries/urdf/legacy/gripper_new.xacro (robot description, xacro)
@@ -158,5 +158,5 @@
                     rpy="0 0 0" />
             <geometry>
-                <mesh filename="${mesh_location}/gripper/gripper_base.stl" />
+                <mesh filename="${mesh_location}/unused/gripper/gripper_base.stl" />
             </geometry>
             <material
@@ -169,5 +169,5 @@
                     rpy="0 0 0" />
             <geometry>
-                <mesh filename="${mesh_location}/gripper/gripper_base.stl" />
+                <mesh filename="${mesh_location}/unused/gripper/gripper_base.stl" />
             </geometry>
         </collision>
@@ -183,5 +183,5 @@
             <origin xyz="0 0 0" rpy="0 0 0" />
             <geometry>
-                <mesh filename="${mesh_location}/gripper/gripper_base_pins.stl" />
+                <mesh filename="${mesh_location}/unused/gripper/gripper_base_pins.stl" />
             </geometry>
             <material name="">
@@ -198,5 +198,5 @@
                     rpy="0 0 0" />
             <geometry>
-                <mesh filename="${mesh_location}/gripper/gripper_gear_left.stl" />
+                <mesh filename="${mesh_location}/unused/gripper/gripper_gear_left.stl" />
             </geometry>
             <material
@@ -209,5 +209,5 @@
                     rpy="0 0 0" />
             <geometry>
-                <mesh filename="${mesh_location}/gripper/gripper_gear_left.stl" />
+                <mesh filename="${mesh_location}/unused/gripper/gripper_gear_left.stl" />
             </geometry>
         </collision>
@@ -221,5 +221,5 @@
             <origin xyz="0 0 0" rpy="0 0 0" />
             <geometry>
-                <mesh filename="${mesh_location}/gripper/gripper_gear_left_plate2.stl" />
+                <mesh filename="${mesh_location}/unused/gripper/gripper_gear_left_plate2.stl" />
             </geometry>
             <material name="">
@@ -244,5 +244,5 @@
                     rpy="0 0 0" />
             <geometry>
-                <mesh filename="${mesh_location}/gripper/gripper_gear_right.stl" />
+                <mesh filename="${mesh_location}/unused/gripper/gripper_gear_right.stl" />
             </geometry>
             <material
@@ -255,5 +255,5 @@
                     rpy="0 0 0" />
             <geometry>
-                <mesh filename="${mesh_location}/gripper/gripper_gear_right.stl" />
+                <mesh filename="${mesh_location}/unused/gripper/gripper_gear_right.stl" />
             </geometry>
         </collision>
@@ -262,5 +262,5 @@
             <origin xyz="0 0 0" rpy="0 0 0" />
             <geometry>
-                <mesh filename="${mesh_location}/gripper/gripper_gear_right_plate2.stl" />
+                <mesh filename="${mesh_location}/unused/gripper/gripper_gear_right_plate2.stl" />
             </geometry>
             <material name="">
@@ -286,5 +286,5 @@
                     rpy="0 0 0" />
             <geometry>
-                <mesh filename="${mesh_location}/gripper/gripper_link_left.stl" />
+                <mesh filename="${mesh_location}/unused/gripper/gripper_link_left.stl" />
             </geometry>
             <material
@@ -297,5 +297,5 @@
                     rpy="0 0 0" />
             <geometry>
-                <mesh filename="${mesh_location}/gripper/gripper_link_left.stl" />
+                <mesh filename="${mesh_location}/unused/gripper/gripper_link_left.stl" />
             </geometry>
         </collision>
@@ -304,5 +304,5 @@
             <origin xyz="0 0 0" rpy="0 0 0" />
             <geometry>
-                <mesh filename="${mesh_location}/gripper/gripper_link_left_plate2.stl" />
+                <mesh filename="${mesh_location}/unused/gripper/gripper_link_left_plate2.stl" />
             </geometry>
             <material name="">
@@ -347,5 +347,5 @@
                     rpy="0 0 0" />
             <geometry>
-                <mesh filename="${mesh_location}/gripper/gripper_link_right.stl" />
+                <mesh filename="${mesh_location}/unused/gripper/gripper_link_right.stl" />
             </geometry>
             <material
@@ -358,5 +358,5 @@
                     rpy="0 0 0" />
             <geometry>
-                <mesh filename="${mesh_location}/gripper/gripper_link_right.stl" />
+                <mesh filename="${mesh_location}/unused/gripper/gripper_link_right.stl" />
             </geometry>
         </collision>
@@ -365,5 +365,5 @@
             <origin xyz="0 0 0" rpy="0 0 0" />
             <geometry>
-                <mesh filename="${mesh_location}/gripper/gripper_link_right_plate2.stl" />
+                <mesh filename="${mesh_location}/unused/gripper/gripper_link_right_plate2.stl" />
             </geometry>
             <material name="">
@@ -409,5 +409,5 @@
                     rpy="0 0 0" />
             <geometry>
-                <mesh filename="${mesh_location}/gripper/${finger_mesh}" />
+                <mesh filename="${mesh_location}/unused/gripper/${finger_mesh}" />
             </geometry>
             <material
@@ -475,5 +475,5 @@
                     rpy="0 0 0" />
             <geometry>
-                <mesh filename="${mesh_location}/gripper/${finger_mesh}" />
+                <mesh filename="${mesh_location}/unused/gripper/${finger_mesh}" />
             </geometry>
             <material
@@ -592,4 +592,4 @@
     </joint>
     <!-- Gripper Camera (D435i) — defined in gripper_camera.xacro -->
-    <xacro:include filename="gripper_camera.xacro" />
+    <xacro:include filename="$(find aries)/urdf/gripper_camera.xacro" />
 </robot>

File: src/aries/urdf/legacy/gripper_standalone.urdf.xacro (robot description, xacro)
@@ -23,4 +23,4 @@
     </joint>
     <!-- Include gripper xacro (it will attach to link6) -->
-    <xacro:include filename="$(find aries)/urdf/gripper.xacro"/>
+    <xacro:include filename="$(find aries)/urdf/legacy/gripper.xacro"/>
 </robot>

File: src/aries/urdf/legacy/gripper_with_arduino_control.urdf.xacro (robot description, xacro)
@@ -29,5 +29,5 @@
     </joint>
     <!-- Include gripper xacro (it will attach to link6) -->
-    <xacro:include filename="$(find aries)/urdf/gripper.xacro"/>
+    <xacro:include filename="$(find aries)/urdf/legacy/gripper.xacro"/>
     <!-- ros2_control using Teensy hardware -->
     <ros2_control name="TeensyGripperHardware" type="system">

File: src/aries/urdf/legacy/gripper_with_mock_control.urdf.xacro (robot description, xacro)
@@ -27,5 +27,5 @@
     </joint>
     <!-- Include gripper xacro (it will attach to link6) -->
-    <xacro:include filename="$(find aries)/urdf/gripper.xacro"/>
+    <xacro:include filename="$(find aries)/urdf/legacy/gripper.xacro"/>
     <!-- ros2_control using mock hardware -->
     <ros2_control name="GripperMockHardware" type="system">

File: src/aries/urdf/my_robot.urdf.xacro (robot description, xacro)
@@ -1,9 +1,13 @@
 <?xml version="1.0"?>
 <robot xmlns:xacro="http://www.ros.org/wiki/xacro" name="aries">
-  <!-- Gripper selection - 'v2' (REBEL-6DOF-04, meshing sector gears),
-       'new' (the 85.563 mm four-bar) or 'old' -->
+  <!-- The REBEL-6DOF-04 gripper (meshing sector gears) is the only gripper
+       this robot is built with. The 85.563 mm four-bar ('new') and the
+       original ('old') are retired to urdf/legacy/ and are not reachable from
+       here; nothing in the fleet runs them any more.
+       The argument is still declared because a dozen launch files pass
+       gripper_type:=v2 down to this file, and an undeclared arg is a hard
+       error. It is accepted and ignored - there is no branch left to take. -->
   <xacro:arg name="gripper_type" default="v2"/>
-  <xacro:property name="gripper_type" value="$(arg gripper_type)"/>
-  <!-- Swappable fingertip - 'bucket', 'maintenance', or 'probe' (new gripper only) -->
+  <!-- Swappable fingertip - 'bucket', 'maintenance', or 'probe' -->
   <xacro:arg name="finger_type" default="probe"/>
   <xacro:property name="finger_type" value="$(arg finger_type)"/>
@@ -22,4 +26,5 @@
   <xacro:include filename="aries_gazebo.xacro"/>
   <xacro:include filename="aries_base.xacro"/>
+  <xacro:include filename="drill.xacro"/>
   <xacro:include filename="differential_link.xacro"/>
   <xacro:include filename="left_link.xacro"/>
@@ -31,13 +36,4 @@
   <!-- Instantiate the arm control macro -->
   <xacro:igus_rebel_control arm_id="aries" hardware_protocol="${hardware_protocol}" arm_hardware_protocol="${arm_hardware_protocol}" gripper_hardware_protocol="${gripper_hardware_protocol}" serial_port="${serial_port}"/>
-  <!-- Conditional gripper includes -->
-  <xacro:if value="${gripper_type == 'v2'}">
-    <xacro:include filename="gripper_v2.xacro"/>
-  </xacro:if>
-  <xacro:if value="${gripper_type == 'new'}">
-    <xacro:include filename="gripper_new.xacro"/>
-  </xacro:if>
-  <xacro:if value="${gripper_type == 'old'}">
-    <xacro:include filename="gripper.xacro"/>
-  </xacro:if>
+  <xacro:include filename="gripper_v2.xacro"/>
 </robot>

File: src/aries/urdf/rover.urdf.xacro (robot description, xacro)
@@ -5,4 +5,5 @@
   <xacro:include filename="aries_gazebo.xacro"/>
   <xacro:include filename="aries_base.xacro"/>
+  <xacro:include filename="drill.xacro"/>
   <xacro:include filename="differential_link.xacro"/>
   <xacro:include filename="left_link.xacro"/>
